File: sim-monitor-sd/_autosave-sim-monitor-sd.kicad_pcb (KiCad board)
At the start: 2 copper layers, 29 parts, among them J1 A-DF_09_A_KG-T4S, U1 ESP32-DEVKITC-32D, U2 LTV-846S, U4 MP2315SGJ-Z

Commit message: pcb update
Parts:
- moved R10 10.5 mm to (75.0, 65.0), turned to 180 degrees
- moved C1 6.50 mm to (75.0, 59.5)
- moved C2 5.50 mm to (75.0, 55.0)
Connections:
- R9 pad 1: GND -> Net-(U1-IO17)
- R9 pad 2: Net-(U1-IO17) -> GND
Routing:
- net +24V: track 0.00 -> 306.7 mm, vias 0 -> 5
- net GND: track 0.00 -> 200.0 mm, vias 0 -> 2
- net Net-(U1-IO2): track 0.00 -> 84.0 mm, vias 0 -> 1
- net +5V: track 0.00 -> 80.2 mm, vias 0 -> 1
- net Net-(U1-IO4): track 0.00 -> 79.3 mm, vias 0 -> 1
- net Net-(U1-IO17): track 0.00 -> 71.9 mm, vias 0 -> 2
- net Net-(U1-IO16): track 0.00 -> 71.5 mm, vias 0 -> 1
- net +3.3V: track 0.00 -> 68.8 mm
- net Net-(C5-Pad1): track 0.00 -> 43.4 mm, vias 0 -> 2
- net Net-(U1-IO25): track 0.00 -> 34.2 mm, vias 0 -> 1
- net Net-(U1-IO26): track 0.00 -> 33.6 mm, vias 0 -> 1
- net Net-(U1-IO27): track 0.00 -> 29.5 mm, vias 0 -> 1
- net Net-(U4-EN): track 0.00 -> 27.5 mm, vias 0 -> 2
- net Net-(U1-IO14): track 0.00 -> 25.3 mm
- net Net-(U4-SW): track 0.00 -> 21.6 mm
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Other:
- board outline added: 84 x 67 mm
