File: sim-monitor-sd/final-pcb.kicad_pcb (KiCad board)
At the start: 2 copper layers, 84 x 67 mm, 29 parts, among them J1 A-DF_09_A_KG-T4S, U1 ESP32-DEVKITC-32D, U2 LTV-846S, U4 MP2315SGJ-Z

Commit message: pcb update
Routing:
- net +5V: track 80.2 -> 47.3 mm, vias 1 -> 0
- net Net-(C5-Pad1): track 43.4 -> 41.5 mm
- net +24V: track 306.7 -> 307.3 mm
- net Net-(R12-Pad2): track 13.6 -> 14.2 mm

Commit message: pcb update
Parts:
- added ?: , , F.Cu at (113.6, 70.6)
- added ?: , , F.Cu at (108.6, 70.6)
- moved D1 2.00 mm to (109.0, 79.5)
Routing:
- net +24V: track 307.3 -> 326.0 mm, vias 5 -> 7
- net +5V: track 47.3 -> 56.6 mm
- net Net-(C5-Pad1): track 41.5 -> 45.5 mm
- net Net-(U4-SW): track 21.6 -> 25.5 mm
- net GND: track 199.7 -> 197.8 mm
- net Net-(R12-Pad2): track 14.2 -> 13.0 mm
- net Net-(U1-IO25): track 34.2 -> 34.8 mm
- added copper zone on B.Cu, net GND
- added copper zone on F.Cu, net GND
Other:
- board size 84 x 67 mm -> 87 x 67 mm
- board text added: "CHUCHU Alexsandr.Chuchupalov@FlightSafety.com"
- board text added: "Christopher Francis christopher.francis@FlightSafety.com"
- board text added: "Demetrius M7 Ross Demetrius.Ross@FlighSafety.com"
- board text added: "ESP Sender board for Sim Monitor project"
- board text added: "Sim ESP Sender Module Mk 1"
