File: sim-monitor-sd/sim-monitor-sd.kicad_sch (KiCad schematic)
At the start: 1 part, among them U1 ESP32-DEVKITC-32D

Commit message: sd
Parts:
- added C1: CL31A226KAHNNNE, CL31A226KAHNNNE:CAPC3216X180N, symbol CL31A226KAHNNNE:CL31A226KAHNNNE
- added C2: CL31B106KAHNNNE, CL31B106KAHNNNE:CAPC3216X180N, symbol CL31B106KAHNNNE:CL31B106KAHNNNE
- added C3, C4: C1206C104K4RACTU, C1206C104K4RACTU:CAPC3216X88N, symbol C1206C104K4RACTU:C1206C104K4RACTU
- added D1: SS14, Diode_SMD:D_SMA, symbol Diode:SS14
- added R1, R2, R3: CR1206-FX-1002ELF, CR1206-FX-1002ELF:RESC3216X75N, symbol CR1206-FX-1002ELF:CR1206-FX-1002ELF
- added R4, R5, R6: CR1206-FX-2200ELF, CR1206-FX-2200ELF:RESC3216X75N, symbol CR1206-FX-2200ELF:CR1206-FX-2200ELF
- added R7, R8, R9: CR1206-FX-4700ELF, CR1206-FX-4700ELF:RESC3216X75N, symbol CR1206-FX-4700ELF:CR1206-FX-4700ELF
- added S1: DRR3016, DRR3016:DRR3010, symbol DRR3016:DRR3016
- added U2, U3: TLP291-4, Package_SO:SOIC-16_4.55x10.3mm_P1.27mm, symbol Isolator:TLP291-4
- added U4: MP2315SGJ-Z, TSOT23-8_MP2315S_MNP, symbol 2025-03-04_06-48-30:MP2315SGJ-Z

Commit message: 3Mar
Parts:
- added J1: A-DF_09_A_KG-T4S, A-DF_09_A_KG-T4S:ASSMANN_A-DF_09_A_KG-T4S, symbol A-DF_09_A_KG-T4S:A-DF_09_A_KG-T4S
Connections:
- net +5V: now reaches U4.7 (VCC)
- new net +24V: J1.1
Other:
- moved on the sheet: C1, C2, C3, C4, D1, R1, R2, R3, R4, R5, R6, R7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

Commit message: 6Mar
Parts:
- removed C2: CL31B106KAHNNNE, CL31B106KAHNNNE:CAPC3216X180N, symbol CL31B106KAHNNNE:CL31B106KAHNNNE
- added C5, C6: CL31A226KAHNNNE, CL31A226KAHNNNE:CAPC3216X180N, symbol CL31A226KAHNNNE:CL31A226KAHNNNE
- added L1: HPC6045NC-4R7M, IND_HPC6045NC_TTA, symbol 2025-03-06_05-32-12:HPC6045NC-4R7M
- added R10: RC1206FR-07499KL, RC1206FR-07499KL:RESC3116X65N, symbol RC1206FR-07499KL:RC1206FR-07499KL
- added R11: RMCF1206FT10R0, RMCF1206FT10R0:RESC3216X70N, symbol RMCF1206FT10R0:RMCF1206FT10R0
- added R12: RMCF1206FT40K2, RMCF1206FT40K2:RESC3216X70N, symbol RMCF1206FT40K2:RMCF1206FT40K2
- added R13: RMCF1206FT7K50, RMCF1206FT7K50:RESC3216X70N, symbol RMCF1206FT7K50:RMCF1206FT7K50
- added R14: CRCW120620K0FKEAC, CRCW120620K0FKEAC:RESC3015X65N, symbol CRCW120620K0FKEAC:CRCW120620K0FKEAC
- added R15: CR1206-FX-1002ELF, CR1206-FX-1002ELF:RESC3216X75N, symbol CR1206-FX-1002ELF:CR1206-FX-1002ELF
Connections:
- net +24V: now also R10.2
- net +5V: now also C5.1, C6.1, L1.1, R12.1; no longer U4.7 (VCC)
- net GND: now also J1.6
- net at U1.J2-19 (EXT_5V): now also D1.1 (K)
- net at U4.2 (IN): now also C1.1, C3.1
- net at U4.3 (SW): now also C4.1, L1.2
- net at U4.4 (GND): now also C1.2, C3.2, U2.6, U2.8, U3.2, U3.4, C5.2, C6.2, R13.1
- net at U4.5 (BST): now also R11.1
- net at U4.6 (EN): now also R10.1
- net at U4.8 (FB): now also R14.2
- net at C4.2: now also R11.2
- net at U3.1: now also R1.2
- net at U2.5: now also R3.2
- net at R2.1: now also J1.4
- net at R2.2: now also U3.3
- net at J1.2: now also R15.1
- net at J1.3: now also R3.1
- net at J1.5: now also R1.1
- net at U2.7: now also R15.2
- new net: R12.2, R13.2, R14.1
Other:
- moved on the sheet: C1, C3, C4, D1, J1, R1, R2, R3, U2C, U2D, U3A, U3B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

Commit message: 7Mar
Parts:
- removed R1, R2, R3: CR1206-FX-1002ELF, CR1206-FX-1002ELF:RESC3216X75N, symbol CR1206-FX-1002ELF:CR1206-FX-1002ELF
- removed R4, R5, R6: CR1206-FX-2200ELF, CR1206-FX-2200ELF:RESC3216X75N, symbol CR1206-FX-2200ELF:CR1206-FX-2200ELF
- removed R7, R8, R9: CR1206-FX-4700ELF, CR1206-FX-4700ELF:RESC3216X75N, symbol CR1206-FX-4700ELF:CR1206-FX-4700ELF
- removed U2, U3: TLP291-4, Package_SO:SOIC-16_4.55x10.3mm_P1.27mm, symbol Isolator:TLP291-4
- added R1, R2, R3, R4: CRGCQ1206F2K2, CRGCQ1206F2K2:RESC3115X65N, symbol CRGCQ1206F2K2:CRGCQ1206F2K2
- added R16, R17, R5, R6, R7, R8, R9: CR1206-FX-1002ELF, CR1206-FX-1002ELF:RESC3216X75N, symbol CR1206-FX-1002ELF:CR1206-FX-1002ELF
- added U2: LTV-846S, LTV-846S:SOIC254P1016X460-16N, symbol LTV-846S:LTV-846S
Connections:
- net +24V: now also J1.2, J1.3, J1.4, J1.5; no longer R10.2
- net GND: now also C1.2, C3.2, C5.2, C6.2, R13.1, R15.2, U1.J2-14 (GND1), U4.4 (GND), R16.2, R17.2, R9.1, U2.2, U2.4, U2.6, U2.8
- net +3.3V: now reaches U1.J2-1 (3V3)
- net at U1.J2-10 (IO26): now also R6.1, U2.11
- net at U1.J2-11 (IO27): now also R7.1, U2.13
- net at U1.J2-12 (IO14): now also R8.1, U2.15
- net at U1.J2-9 (IO25): now also R5.1, U2.9
- net at U1.J3-11 (IO17): now also S1.8, R9.2
- net at U1.J3-12 (IO16): now also R15.1, S1.4
- net at U1.J3-13 (IO4): now also S1.2, R16.1
- net at U1.J3-15 (IO2): now also S1.1, R17.1
- net at C1.1, C3.1, U4.2 (IN): now also R10.2
- net at S1.C: now also R5.2, R6.2, R7.2, R8.2, U2.10, U2.12, U2.14, U2.16
- new net: R3.2, U2.5
- new net: R4.2, U2.7
- new net: R1.2, U2.1
- new net: R2.2, U2.3
Other:
- note added: "ESPNOW-SENDER Board v1"
- moved on the sheet: S1, U1

Commit message: 8Mar
Parts:
- removed D1: SS14, Diode_SMD:D_SMA, symbol Diode:SS14
- added D1: SS34B-HF, SS34B_HF:DO214AASMB_CIP, symbol 2025-03-08_07-44-24:SS34B-HF
- J1: footprint A-DF_09_A_KG-T4S:ASSMANN_A-DF_09_A_KG-T4S -> A_DF_09_A_KG_T4S:ASSMANN_A-DF_09_A_KG-T4S
- L1: footprint IND_HPC6045NC_TTA -> ul_HPC6045NC-4R7M:IND_HPC6045NC_TTA
- R10: footprint RC1206FR-07499KL:RESC3116X65N -> RC1206FR_07499KL:RESC3116X65N
- R15, R16, R17, R5, R6, R7, R8, R9: footprint CR1206-FX-1002ELF:RESC3216X75N -> CR1206_FX_1002ELF:RESC3216X75N
- U2: footprint LTV-846S:SOIC254P1016X460-16N -> LTV_846S:SOIC254P1016X460-16N
- U4: footprint TSOT23-8_MP2315S_MNP -> MP2315SGJ_Z:TSOT23-8_MP2315S_MNP
Connections:
- net +24V: now also C1.1, C3.1, R1.1, R10.2, R2.1, R3.1, R4.1, U4.2 (IN)
- net +3.3V: now also R5.2, R6.2, R7.2, R8.2, S1.C, U2.10, U2.12, U2.14, U2.16
- net +5V: now also R11.1, U1.J2-19 (EXT_5V), U4.5 (BST), D1.1; no longer C5.1, C6.1, L1.1, R12.1
- net GND: now also U1.J3-7 (GND2)
- new net: C5.1, C6.1, D1.2, L1.1, R12.1
- no-connect marks 0 -> 33
Other:
- moved on the sheet: J1, R11, R16, R17

Commit message: pcb update
Parts:
- removed C3, C4: C1206C104K4RACTU, C1206C104K4RACTU:CAPC3216X88N, symbol C1206C104K4RACTU:C1206C104K4RACTU
- added C2, C3: CL31B106KAHNNNE, CL31B106KAHNNNE:CAPC3216X180N, symbol CL31B106KAHNNNE:CL31B106KAHNNNE
Connections:
- net +24V: now also C2.1
- net GND: now also R9.2, C2.2; no longer R9.1
- net at R6.1, U2.11: now also U1.J2-11 (IO27); no longer U1.J2-10 (IO26)
- net at R7.1, U2.13: now also U1.J2-10 (IO26); no longer U1.J2-11 (IO27)
- net at R8.1, U2.15: now also U1.J2-9 (IO25); no longer U1.J2-12 (IO14)
- net at R5.1, U2.9: now also U1.J2-12 (IO14); no longer U1.J2-9 (IO25)
- net at S1.8, U1.J3-11 (IO17): now also R9.1; no longer R9.2
- net at R11.2: now also C3.1
- net at L1.2, U4.3 (SW): now also C3.2
Other:
- moved on the sheet: R9

Commit message: pcb update
Changed lines of the file:
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@@
 		)
 		(property "Value" "CR1206-FX-1002ELF"
-			(at 256.794 100.33 0)
+			(at 256.032 98.044 0)
 			(effects
 				(font
