File: board_design/schematic_V2.kicad_sch (KiCad schematic)
At the start: 26 parts, among them J1 A-DF_09_A_KG-T4S, U1 ESP32-DEVKITC-32D, U2 LTV-846S

Commit message: updated schematic
Parts:
- added C3: 1000pf/3kV, CL31B106KAHNNNE:CAPC3216X180N, symbol CL31B106KAHNNNE:CL31B106KAHNNNE
Connections:
- net GND: now also C3.2
- net at PS1.16 (-VOUT), U1.J3-1 (GND3): now also C3.1
Changed lines of the file:
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@@
 	)
 	(junction
+		(at 115.57 148.59)
+		(diameter 0)
+		(color 0 0 0 0)
+	)
+	(junction
 		(at 167.64 73.66)
 		(diameter 0)
@@
 	(wire
 		(pts
+			(xy 115.57 148.59) (xy 111.76 148.59)
+		)
+		(stroke
+			(width 0)
+			(type default)
+		)
+	)
+	(wire
+		(pts
 			(xy 267.97 24.13) (xy 267.97 26.67)
 		)
@@
 	(wire
 		(pts
+			(xy 115.57 173.99) (xy 115.57 148.59)
+		)
+		(stroke
+			(width 0)
+			(type default)
+		)
+	)
+	(wire
+		(pts
 			(xy 156.21 78.74) (xy 194.31 78.74)
 		)
@@
 	(wire
 		(pts
+			(xy 74.93 173.99) (xy 92.71 173.99)
+		)
+		(stroke
+			(width 0)
+			(type default)
+		)
+	)
+	(wire
+		(pts
+			(xy 74.93 173.99) (xy 74.93 151.13)
+		)
+		(stroke
+			(width 0)
+			(type default)
+		)
+	)
+	(wire
+		(pts
 			(xy 255.27 55.88) (xy 265.43 55.88)
 		)
@@
 	(wire
 		(pts
-			(xy 283.21 148.59) (xy 111.76 148.59)
+			(xy 283.21 148.59) (xy 115.57 148.59)
+		)
+		(stroke
+			(width 0)
+			(type default)
+		)
+	)
+	(wire
+		(pts
+			(xy 100.33 173.99) (xy 115.57 173.99)
 		)
 		(stroke
@@
 	)
 	(symbol
+		(lib_id "CL31B106KAHNNNE:CL31B106KAHNNNE")
+		(at 95.25 173.99 0)
+		(unit 1)
+		(exclude_from_sim no)
+		(in_bom yes)
+		(on_board yes)
+		(dnp no)
+		(fields_autoplaced yes)
+		(property "Reference" "C3"
+			(at 96.52 167.64 0)
+			(effects
+				(font
+					(size 1.27 1.27)
+				)
+			)
+		)
+		(property "Value" "1000pf/3kV"
+			(at 96.52 170.18 0)
+			(effects
+				(font
+					(size 1.27 1.27)
+				)
+			)
+		)
+		(property "Footprint" "CL31B106KAHNNNE:CAPC3216X180N"
+			(at 95.25 173.99 0)
+			(effects
+				(font
+					(size 1.27 1.27)
+				)
+				(justify bottom)
+				(hide yes)
+			)
+		)
+		(property "Datasheet" ""
+			(at 95.25 173.99 0)
+			(effects
+				(font
+					(size 1.27 1.27)
+				)
+				(hide yes)
+			)
+		)
+		(property "Description" ""
+			(at 95.25 173.99 0)
+			(effects
+				(font
+					(size 1.27 1.27)
+				)
+				(hide yes)
+			)
+		)
+		(pin "1"
+		)
+		(pin "2"
+		)
+		(instances
+			(project ""
+				(path "/1521a3d4-d148-4383-b633-021e5ea56970"
+					(reference "C3")
+					(unit 1)
+				)
+			)
+		)
+	)
+	(symbol
 		(lib_id "CR1206-FX-1002ELF:CR1206-FX-1002ELF")
 		(at 184.15 31.75 90)
@@
 		)
 		(property "Value" "UHE2A470MPD"
-			(at 63.5 140.716 90)
+			(at 69.596 140.716 90)
 			(effects
 				(font
@@
 		(dnp no)
 		(property "Reference" "C2"
-			(at 74.93 154.178 90)
+			(at 74.93 138.176 90)
 			(effects
 				(font
@@
 					(size 1.524 1.524)
 				)
+				(hide yes)
 			)
 		)
