File: board_design/schematic_Mk2.kicad_sch (KiCad schematic)
At the start: 29 parts, among them J1 A-DF_09_A_KG-T4S, J2 1757255, SW1 On/Off Switch, U1 ESP32-DEVKITC-32D, U2 LTV-846S

Commit message: updated
Parts:
- RF1, RF2: footprint footprints:PCAP_10x12_5-THRU-ELECT_NCA -> footprints:PTC_RESET_FUSE
Changed lines of the file:
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@@
 			)
 		)
-		(property "Footprint" "footprints:PCAP_10x12_5-THRU-ELECT_NCA"
+		(property "Footprint" "footprints:PTC_RESET_FUSE"
 			(at 179.07 148.59 0)
 			(effects
@@
 			)
 		)
-		(property "Footprint" "footprints:PCAP_10x12_5-THRU-ELECT_NCA"
+		(property "Footprint" "footprints:PTC_RESET_FUSE"
 			(at 100.33 148.59 0)
 			(effects
