File: board_design/schematic_Mk2.1.kicad_pcb (KiCad board)
At the start: 2 copper layers, 29 parts, among them J1 A-DF_09_A_KG-T4S, J2 1757255, SW1 On/Off Switch, U1 ESP32-DEVKITC-32D, U2 LTV-846S

Commit message: pcb update
Parts:
- added J3: JCT, footprints:CONN_BM04B-SRSS-TB_SPK, F.Cu at (196.5, 85.5)
- C3, D1, R1, R10, R11, R12, R13, R14, R15, R16, R2, R3, R4, R5, R6, R7, R8, R9: moved to B.Cu
- moved R16 120.6 mm to (192.0, 75.0), turned to 180 degrees
- moved R13 120.6 mm to (192.0, 65.0), turned to 180 degrees
- moved R15 120.5 mm to (192.0, 70.0), turned to 180 degrees
- moved R14 120.4 mm to (192.0, 60.0), turned to 180 degrees
- moved R9 117.5 mm to (189.0, 37.5)
- moved R12 117.5 mm to (189.0, 47.5)
- moved R10 117.5 mm to (189.0, 42.5)
- moved R11 117.4 mm to (189.0, 53.0)
- moved U2 115.0 mm to (159.5, 44.1)
- moved RF2 87.9 mm to (179.0, 86.0)
- moved C1 73.6 mm to (147.3, 75.1), turned to 180 degrees
- moved S1 72.8 mm to (159.2, 28.5), turned to 180 degrees
- moved PS1 69.1 mm to (163.4, 73.0), turned to -90 degrees
- moved C2 68.6 mm to (147.3, 64.1), turned to 180 degrees
- moved J2 68.2 mm to (124.5, 61.2)
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Connections:
- R16 pad 1: GPIO_4 -> GPIO_2
- U1 pad J3-3: unconnected-(U1-IO22-PadJ3-3) -> GPIO_22
- U1 pad J3-6: unconnected-(U1-IO21-PadJ3-6) -> GPIO_21
Other:
- board outline added: 81.2 x 68 mm
- rule pad_to_mask_clearance: 0 -> 0.0508
