File: board_design/schematic_Mk2.1.kicad_pcb (KiCad board)
At the start: 2 copper layers, 82.8 x 74 mm, 32 parts, among them J1 A-DF_09_A_KG-T4S, J2 1757255, J3 JST -SM, J4 S3B-EH, U1 ESP32-DEVKITC-32D, U2 LTV-846S

Commit message: update
Parts:
- R1, R2, R5, R6, U2: moved to B.Cu
- moved J3 69.8 mm to (134.8, 88.6)
- moved C3 51.4 mm to (128.2, 119.1), turned to -90 degrees
- moved RF1 45.8 mm to (111.5, 120.1), turned to 90 degrees
- moved R17 41.9 mm to (163.2, 70.9)
- moved R16 41.4 mm to (163.2, 121.1)
- moved U2 41.4 mm to (136.2, 72.3)
- moved J2 41.3 mm to (95.7, 105.9)
- moved R18 41.1 mm to (163.2, 64.6)
- moved R15 41.1 mm to (163.2, 114.8)
- moved R5 41.0 mm to (119.2, 82.3)
- moved R6 41.0 mm to (119.2, 86.8)
- moved D1 41.0 mm to (100.5, 109.6)
- moved PS1 41.0 mm to (131.3, 112.6)
- moved R2 41.0 mm to (122.2, 68.1)
- moved R3 41.0 mm to (120.1, 72.6)
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Connections:
- C3 pad 1: -VOUT -> ESP_GND2
- PS1 pad 16: -VOUT -> ESP_GND2
- U1 pad J3-1: -VOUT -> ESP_GND2
- U2 pad 1: Net-(R1-Pad2) -> Net-(R7-Pad2)
- U2 pad 10: GPIO_26 -> GPIO_32
- U2 pad 12: GPIO_25 -> GPIO_33
- U2 pad 14: GPIO_33 -> GPIO_25
- U2 pad 16: GPIO_32 -> GPIO_26
- U2 pad 3: Net-(R3-Pad2) -> Net-(R5-Pad2)
- U2 pad 5: Net-(R5-Pad2) -> Net-(R3-Pad2)
- U2 pad 7: Net-(R7-Pad2) -> Net-(R1-Pad2)
Routing:
- net +3.3V: track 111.1 -> 0.84 mm, vias 2 -> 0
- net GPIO_5: track 88.3 -> 0.30 mm
- net GPIO_17: track 82.0 -> 0.00 mm
- net GPIO_16: track 77.8 -> 0.00 mm
- net GPIO_4: track 71.6 -> 0.00 mm
- net ESP_GND2: track 58.8 -> 0.00 mm
- net GPIO_21: track 36.1 -> 0.00 mm
- net GPIO_22: track 29.0 -> 0.00 mm
- added copper zone on B.Cu, net +VOUT
- added copper zone on F.Cu, net +VOUT
- added copper zone on B.Cu, net spare
- removed copper zone on B.Cu, net sim_home
- removed copper zone on F.Cu, net sim_home
Other:
- board size 82.8 x 74 mm -> 83 x 74.2 mm

Commit message: update
Parts:
- moved J3 29.5 mm to (163.0, 80.1), turned to 180 degrees
- moved R18 22.7 mm to (159.2, 86.9)
- moved R9 17.4 mm to (166.4, 94.3), turned to -90 degrees
- moved R17 16.5 mm to (167.0, 86.9)
- moved R12 14.6 mm to (159.2, 103.7), turned to 90 degrees
- moved J4 13.3 mm to (114.1, 98.7), turned to 0 degrees
- moved D1 12.0 mm to (112.0, 106.0)
- moved R10 11.5 mm to (159.2, 94.2), turned to -90 degrees
- moved C3 11.3 mm to (137.8, 113.0)
- moved R14 10.4 mm to (159.2, 111.8), turned to -90 degrees
- moved R11 8.43 mm to (166.4, 103.8), turned to 90 degrees
- moved R2 7.37 mm to (120.0, 61.0), turned to -90 degrees
- moved R8 7.31 mm to (121.5, 92.5), turned to 45 degrees
- moved R5 6.25 mm to (122.5, 77.0)
- moved R6 6.25 mm to (122.5, 81.5)
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Connections:
- net Net-(R1-Pad2) renamed spare_opto
- net Net-(R3-Pad2) renamed ramp_up_opto
- net Net-(R5-Pad2) renamed /ramp_down_opto
- net Net-(R7-Pad2) renamed /sim_home_opto
- C1 pad 1: Net-(PS1-+VIN) -> +24V
- C2 pad 1: Net-(PS1-+VIN) -> +24V
- D1 pad 2: Net-(D1-Pad2) -> +24V
- J2 pad 02: Net-(D1-Pad2) -> +24V
- J4 pad 2: +VIN -> +24V
- PS1 pad 14: Net-(PS1-+VOUT) -> +VOUT
- PS1 pad 22: Net-(PS1-+VIN) -> +24V
- RF1 pad 1: +VIN -> +24V
- RF1 pad 2: Net-(PS1-+VIN) -> +24V
- RF2 pad 1: Net-(PS1-+VOUT) -> +VOUT
Routing:
- net +3.3V: track 0.84 -> 146.6 mm, vias 0 -> 2
- net ESP_GND2: track 0.00 -> 70.8 mm, vias 0 -> 1
- net GPIO_5: track 0.30 -> 55.5 mm
- net GPIO_16: track 0.00 -> 53.6 mm
- net GPIO_17: track 0.00 -> 42.2 mm, vias 0 -> 2
- net GPIO_22: track 0.00 -> 39.3 mm
- net GPIO_4: track 0.00 -> 37.4 mm, vias 0 -> 1
- net GPIO_26: track 0.00 -> 32.8 mm, vias 0 -> 1
- net GPIO_21: track 0.00 -> 32.8 mm
- net GPIO_25: track 0.00 -> 28.6 mm, vias 0 -> 1
- net GPIO_32: track 0.00 -> 22.9 mm, vias 0 -> 1
- net GPIO_33: track 0.00 -> 15.6 mm, vias 0 -> 1
- net spare: vias 0 -> 11
- net ramp_up: vias 0 -> 9
- net ramp_down: vias 18 -> 9
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- added copper zone on B.Cu, net +24V
- added copper zone on F.Cu, net +24V
- added copper zone on B.Cu, net -Vin
- added copper zone on B.Cu, net /ramp_down_opto
- added copper zone on F.Cu, net /ramp_down_opto
- added copper zone on B.Cu, net /sim_home_opto
- added copper zone on F.Cu, net /sim_home_opto
- added copper zone on B.Cu, net ESP_GND2
- added copper zone on F.Cu, net ESP_GND2
- added copper zone on B.Cu, net GPIO_25
- added copper zone on B.Cu, net GPIO_26
- added copper zone on B.Cu, net GPIO_32
- added copper zone on B.Cu, net GPIO_33
- added copper zone on B.Cu, net ramp_up_opto
- added copper zone on F.Cu, net ramp_up_opto
- added copper zone on B.Cu, net sim_home
- added copper zone on F.Cu, net sim_home
- added copper zone on B.Cu, net spare_opto
- added copper zone on F.Cu, net spare_opto
Other:
- board size 83 x 74.2 mm -> 83 x 77.2 mm
