File: board_design/schematic_Mk2.1.kicad_pcb (KiCad board)
At the start: 2 copper layers, 83.4 x 77.2 mm, 33 parts, among them J1 A-DF_09_A_KG-T4S, J2 jst-power, J3 JST -SM, J4 S3B-EH, J5 1770979, U1 ESP32-DEVKITC-32D, U2 LTV-846S

Commit message: board update
Other:
- board text added: "Demetrius Ross Demetrius.Ross@flightsafety.com Christopher Francis Christopher.Francis@flightsafety.com ChuChu Alexsandr.Chuchupalov@flightsafety.com"
- board text added: "Mark III"
- board text removed: "Demetrius Ross Demetrius.Ross@flightsafety.com Christopher Francis Christopher.Francis@flightsafety.com Chu Chu Alexsandr.Chuchupalov@flightsafety.com"
- board text removed: "Mark II"
Changed lines of the file:
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@@
 			(outputformat 1)
 			(mirror no)
-			(drillshape 1)
+			(drillshape 0)
 			(scaleselection 1)
-			(outputdirectory "")
+			(outputdirectory "gerber_files/")
 		)
 	)
@@
 		(layer "Edge.Cuts")
 	)
-	(gr_text "Mark II"
+	(gr_text "Mark III"
 		(at 154.8 124.2 0)
 		(layer "F.SilkS")
@@
 		)
 	)
-	(gr_text "Demetrius Ross\nDemetrius.Ross@flightsafety.com\n\n\nChristopher Francis\nChristopher.Francis@flightsafety.com\n\n\nChu Chu\nAlexsandr.Chuchupalov@flightsafety.com"
+	(gr_text "Demetrius Ross\nDemetrius.Ross@flightsafety.com\n\n\nChristopher Francis\nChristopher.Francis@flightsafety.com\n\n\nChuChu\nAlexsandr.Chuchupalov@flightsafety.com"
 		(at 128.365 88.4 0)
 		(layer "F.SilkS")
@@
 		(polygon
 			(pts
-				(xy 123.5 93.5) (xy 116.5 86.5) (xy 118.625 84.8) (xy 127.3875 84.8) (xy 127.3875 84.8) (xy 132.45 84.8)
-				(xy 132.45 87.2) (xy 128.81818 87.2) (xy 128 89)
+				(xy 123.5 93.5) (xy 116.5 86.5) (xy 118.625 84.8) (xy 127.3875 84.8) (xy 132.45 84.8) (xy 132.45 87.2)
+				(xy 128.81818 87.2) (xy 128 89)
 			)
 		)
