File: board_design/_autosave-schematic_Mk2.1.kicad_pcb (KiCad board)
At the start: 2 copper layers, 82.8 x 74 mm, 32 parts, among them J1 A-DF_09_A_KG-T4S, J2 1757255, J3 JST -SM, J4 S3B-EH, U1 ESP32-DEVKITC-32D, U2 LTV-846S

Commit message: pcb update
Parts:
- moved RF1 6.00 mm to (139.0, 89.5), turned to 90 degrees
- moved C3 0.25 mm to (163.0, 81.5)
- turned R10 to 180 degrees
- turned R11 to 180 degrees
- turned R12 to 180 degrees
- turned R9 to 180 degrees
Connections:
- C1 pad 1: Net-(PS1-+VIN) -> +VIN
- C2 pad 1: Net-(PS1-+VIN) -> +VIN
- C3 pad 1: -VOUT -> ESP_GND2
- PS1 pad 14: Net-(PS1-+VOUT) -> +VOUT
- PS1 pad 16: -VOUT -> ESP_GND2
- PS1 pad 22: Net-(PS1-+VIN) -> +VIN
- RF1 pad 2: Net-(PS1-+VIN) -> +VIN
- RF2 pad 1: Net-(PS1-+VOUT) -> +VOUT
Routing:
- net -Vin: track 0.00 -> 63.2 mm, vias 0 -> 1
- net +VIN: track 0.00 -> 32.5 mm
- net +24V: track 0.00 -> 14.3 mm
- net Net-(D1-Pad2): track 0.00 -> 7.14 mm
- added copper zone on B.Cu, net +3.3V
- added copper zone on B.Cu, net +VOUT
- added copper zone on F.Cu, net +VOUT
- added copper zone on B.Cu, net -Vin
- added copper zone on F.Cu, net -Vin
- added copper zone on B.Cu, net ESP_GND2
- added copper zone on F.Cu, net ESP_GND2
- added copper zone on B.Cu, net spare
