File: board_design/schematic_Mk2.1.kicad_sch (KiCad schematic)
At the start: 29 parts, among them J1 A-DF_09_A_KG-T4S, J2 1757255, SW1 On/Off Switch, U1 ESP32-DEVKITC-32D, U2 LTV-846S

Commit message: PCB updated
Parts:
- removed C1, C2: UHE2A470MPD, footprints:PCAP_10x12_5-THRU-ELECT_NCA, symbol 2025-04-04_11-54-12:UHE2A470MPD
- removed D1: SS34B-HF, footprints:DO214AASMB_CIP-L, symbol 2025-03-08_07-44-24:SS34B-HF
- removed J1: A-DF_09_A_KG-T4S, footprints:ASSMANN_A-DF_09_A_KG-T4S, symbol A-DF_09_A_KG-T4S:A-DF_09_A_KG-T4S
- removed PS1: REC5A-2405SW_H2, footprints:CONV_REC5A-2405SW_H2, symbol REC5A-2405SW_H2:REC5A-2405SW_H2
- removed SW1: On/Off Switch, Button_Switch_SMD:Panasonic_EVQPUJ_EVQPUA, symbol Switch:SW_DPST_x2
- removed U1: ESP32-DEVKITC-32D, footprints:MODULE_ESP32-DEVKITC-32D, symbol ESP32-DEVKITC-32D:ESP32-DEVKITC-32D
- added C1, C2: UHE2A470MPD, footprints:PCAP_10x12_5-THRU-ELECT_NCA, symbol custom_library:UHE2A470MPD
- added D1: SS34B-HF, footprints:DO214AASMB_CIP-L, symbol custom_library:SS34B-HF
- added J1: A-DF_09_A_KG-T4S, footprints:ASSMANN_A-DF_09_A_KG-T4S, symbol custom_library:A-DF_09_A_KG-T4S
- added PS1: REC5A-2405SW_H2, footprints:CONV_REC5A-2405SW_H2, symbol custom_library:REC5A-2405SW_H2
- added SW1: On/Off Switch, footprints:SW, symbol custom_library:SW_SPST
- added U1: ESP32-DEVKITC-32D, footprints:MODULE_ESP32-DEVKITC-32D, symbol custom_library:ESP32-DEVKITC-32D
- renumbered R6 to R10, R8 to R11, R7 to R12, R15 to R13, R9 to R14, R16 to R15, R17 to R16, R10 to R5, R11 to R6, R12 to R7, R13 to R8, R5 to R9
Connections:
- net +3.3V: now also U1.J2-1 (3V3)
- net +VIN: now also SW1.2 (B)
- net -Vin: now also C1.2, C2.2, PS1.2 (-VIN)
- net GPIO_14: now also U1.J2-12 (IO14)
- net GPIO_16: now also U1.J3-12 (IO16)
- net GPIO_17: now also U1.J3-11 (IO17)
- net GPIO_2: now also U1.J3-15 (IO2)
- net GPIO_25: now also U1.J2-9 (IO25)
- net GPIO_26: now also U1.J2-10 (IO26)
- net GPIO_27: now also U1.J2-11 (IO27)
- net GPIO_4: now also U1.J3-13 (IO4)
- net -VOUT: now reaches C3.1
- net -VOUT: now also PS1.16 (-VOUT), U1.J3-1 (GND3)
- net at RF2.1: now also PS1.14 (+VOUT)
- net at RF1.2: now also C1.1, C2.1, PS1.22 (+VIN)
- net at RF1.1: now also D1.1
- removed net +24V: R1.1, R2.1, R3.1, R4.1, R5.1, R6.1
- net +5V renamed +VOUT
- net +VOUT: now also U1.J2-19 (EXT_5V)
- net GND renamed ESP_GND
- net ESP_GND: now also U1.J2-14 (GND1); no longer R13.2, R14.2, R15.2, R16.2
- new net: D1.2, SW1.1 (A)
- new net ESP_GND2: R13.2, R14.2, R15.2, R16.2, U1.J3-7 (GND2)
- new net ramp_down: J1.3, R5.1, R6.1
- new net ramp_up: J1.4, R3.1, R4.1
- new net spare: J1.5, R1.1, R2.1
- no-connect marks 36 -> 35

Commit message: pcb update
Parts:
- added J3: JCT, footprints:CONN_BM04B-SRSS-TB_SPK, symbol custom_library:JCT
Connections:
- net +3.3V: now also J3.2
- net ESP_GND2: now also J3.1
- net GPIO_2: now also R16.1
- net GPIO_4: no longer R16.1
- net GPIO_22: now reaches U1.J3-3 (IO22)
- net GPIO_22: now also J3.4
- net GPIO_21: now reaches U1.J3-6 (IO21)
- net GPIO_21: now also J3.3
- no-connect marks 35 -> 33

Commit message: pcb update
Parts:
- removed SW1: On/Off Switch, footprints:SW, symbol custom_library:SW_SPST
- added J4: S3B-EH, footprints:CONN_S3B-EH_JST, symbol custom_library:S3B-EH
- added R17, R18: CR1206-FX-1002ELF, footprints:RESC3216X75N, symbol CR1206-FX-1002ELF:CR1206-FX-1002ELF
- J3: value JCT -> JST -SM
Connections:
- net -VOUT is gone; now on net ESP_GND2: C3.1, PS1.16 (-VOUT), U1.J3-1 (GND3)
- net ESP_GND is gone; now on net ESP_GND2: U1.J2-14 (GND1), U2.11, U2.13, U2.15, U2.9
- net +3.3V: now also R17.1, R18.1
- net +VIN: now also RF1.1, J4.2; no longer J2.02
- net -Vin: now also J2.03, J4.3; no longer J2.01
- net GPIO_16: now also R15.1, S1.2; no longer R13.1, S1.4
- net GPIO_17: now also R13.1, S1.4; no longer R14.1, S1.8
- net GPIO_21: now also R17.2
- net GPIO_22: now also R18.2
- net GPIO_25: now also R12.1, U2.12; no longer R9.1, U2.16
- net GPIO_26: now also R11.1, U2.10; no longer R10.1, U2.14
- net GPIO_4: now also R16.1, S1.1; no longer R15.1, S1.2
- net sim_home: now also J2.01; no longer J2.03
- net +24V: now reaches D1.1
- net +24V: now also J4.1; no longer RF1.1
- net at D1.2: now also J2.02
- net GPIO_32: now reaches U1.J2-7 (IO32)
- net GPIO_32: now also R9.1, U2.16
- net GPIO_33: now reaches U1.J2-8 (IO33)
- net GPIO_33: now also R10.1, U2.14
- net GPIO_5: now reaches U1.J3-10 (IO5)
- net GPIO_5: now also R14.1, S1.8
- removed net GPIO_14: R11.1, U1.J2-12 (IO14), U2.10
- removed net GPIO_2: R16.1, S1.1, U1.J3-15 (IO2)
- removed net GPIO_27: R12.1, U1.J2-11 (IO27), U2.12
Other:
- moved on the sheet: C1, C2, C3, D1, J1, J2, J3, PS1, R13, R14, R15, R16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
