File: board_design/schematic_Mk2.1.kicad_sch (KiCad schematic)
At the start: 32 parts, among them J1 A-DF_09_A_KG-T4S, J2 1757255, J3 JST -SM, J4 S3B-EH, U1 ESP32-DEVKITC-32D, U2 LTV-846S

Commit message: update
Connections:
- net +VIN is gone; now on net +24V: J4.2, RF1.1
- net +24V: now also C1.1, C2.1, D1.2, J2.02, PS1.22 (+VIN), RF1.2
- net +VOUT: now also PS1.14 (+VOUT), RF2.1
- net spare_opto: now reaches R1.2, R2.2, U2.7
- net sim_home_opto: now reaches R7.2, R8.2, U2.1
- net ramp_up_opto: now reaches R3.2, R4.2, U2.5
- net ramp_down_opto: now reaches R5.2, R6.2, U2.3
Other:
- moved on the sheet: RF2
Changed lines of the file:
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@@
 	(wire
 		(pts
-			(xy 191.77 147.32) (xy 194.31 147.32)
+			(xy 195.58 147.32) (xy 198.12 147.32)
 		)
 		(stroke
@@
 	(wire
 		(pts
-			(xy 114.3 74.93) (xy 114.3 67.31)
-		)
-		(stroke
-			(width 0)
-			(type default)
-		)
-	)
-	(wire
-		(pts
 			(xy 90.17 46.99) (xy 90.17 52.07)
 		)
@@
 	(wire
 		(pts
-			(xy 114.3 57.15) (xy 132.08 57.15)
-		)
-		(stroke
-			(width 0)
-			(type default)
-		)
-	)
-	(wire
-		(pts
 			(xy 90.17 24.13) (xy 90.17 29.21)
 		)
@@
 	(wire
 		(pts
+			(xy 120.65 77.47) (xy 120.65 99.06)
+		)
+		(stroke
+			(width 0)
+			(type default)
+		)
+	)
+	(wire
+		(pts
 			(xy 90.17 93.98) (xy 90.17 99.06)
 		)
@@
 	(wire
 		(pts
+			(xy 129.54 57.15) (xy 132.08 57.15)
+		)
+		(stroke
+			(width 0)
+			(type default)
+		)
+	)
+	(wire
+		(pts
 			(xy 87.63 99.06) (xy 90.17 99.06)
 		)
@@
 	(wire
 		(pts
-			(xy 114.3 52.07) (xy 114.3 57.15)
+			(xy 49.53 134.62) (xy 49.53 139.7)
 		)
 		(stroke
@@
 	(wire
 		(pts
-			(xy 120.65 29.21) (xy 120.65 46.99)
+			(xy 90.17 52.07) (xy 90.17 57.15)
 		)
 		(stroke
@@
 	(wire
 		(pts
-			(xy 90.17 52.07) (xy 90.17 57.15)
+			(xy 130.81 147.32) (xy 137.16 147.32)
 		)
 		(stroke
@@
 	(wire
 		(pts
-			(xy 130.81 147.32) (xy 137.16 147.32)
+			(xy 110.49 46.99) (xy 110.49 52.07)
 		)
 		(stroke
@@
 	(wire
 		(pts
-			(xy 110.49 46.99) (xy 110.49 52.07)
+			(xy 110.49 52.07) (xy 110.49 57.15)
 		)
 		(stroke
@@
 	(wire
 		(pts
-			(xy 110.49 52.07) (xy 110.49 57.15)
+			(xy 147.32 46.99) (xy 163.83 46.99)
 		)
 		(stroke
@@
 	(wire
 		(pts
-			(xy 120.65 99.06) (xy 120.65 77.47)
+			(xy 110.49 29.21) (xy 120.65 29.21)
 		)
 		(stroke
@@
 	(wire
 		(pts
-			(xy 147.32 46.99) (xy 163.83 46.99)
+			(xy 163.83 101.6) (xy 176.53 101.6)
 		)
 		(stroke
@@
 	(wire
 		(pts
-			(xy 110.49 29.21) (xy 120.65 29.21)
+			(xy 176.53 40.64) (xy 176.53 57.15)
 		)
 		(stroke
@@
 	(wire
 		(pts
-			(xy 163.83 101.6) (xy 176.53 101.6)
+			(xy 167.64 147.32) (xy 171.45 147.32)
 		)
 		(stroke
@@
 	(wire
 		(pts
-			(xy 176.53 40.64) (xy 176.53 57.15)
+			(xy 114.3 67.31) (xy 114.3 74.93)
 		)
 		(stroke
@@
 		)
 	)
+	(label "+VIN"
+		(at 49.53 138.43 0)
+		(effects
+			(font
+				(size 1.27 1.27)
+			)
+			(justify left bottom)
+		)
+	)
+	(label "-Vin"
+		(at 123.19 154.94 0)
+		(effects
+			(font
+				(size 1.27 1.27)
+			)
+			(justify left bottom)
+		)
+	)
+	(label "ramp_down_opto"
+		(at 114.3 69.85 0)
+		(effects
+			(font
+				(size 1.27 1.27)
+			)
+			(justify left bottom)
+		)
+	)
+	(label "+VOUT"
+		(at 170.18 147.32 90)
+		(effects
+			(font
+				(size 1.27 1.27)
+			)
+			(justify left bottom)
+		)
+	)
+	(label "+VIN"
+		(at 114.3 147.32 0)
+		(effects
+			(font
+				(size 1.27 1.27)
+			)
+			(justify left bottom)
+		)
+	)
+	(label "sim_home_opto"
+		(at 120.65 95.25 0)
+		(effects
+			(font
+				(size 1.27 1.27)
+			)
+			(justify left bottom)
+		)
+	)
+	(label "+VIN"
+		(at 49.53 153.67 0)
+		(effects
+			(font
+				(size 1.27 1.27)
+			)
+			(justify left bottom)
+		)
+	)
 	(global_label "GPIO_32"
 		(shape input)
@@
 		)
 	)
+	(global_label "ramp_up_opto"
+		(shape input)
+		(at 129.54 57.15 180)
+		(fields_autoplaced yes)
+		(effects
+			(font
+				(size 1.27 1.27)
+			)
+			(justify right)
+		)
+		(property "Intersheetrefs" "${INTERSHEET_REFS}"
+			(at 113.3714 57.15 0)
+			(effects
+				(font
+					(size 1.27 1.27)
+				)
+				(justify right)
+				(hide yes)
+			)
+		)
+	)
 	(global_label "GPIO_21"
 		(shape output)
@@
 	(global_label "+24V"
 		(shape output)
-		(at 49.53 139.7 90)
+		(at 49.53 134.62 90)
 		(fields_autoplaced yes)
 		(effects
@@
 		)
 		(property "Intersheetrefs" "${INTERSHEET_REFS}"
-			(at 49.53 131.6348 90)
+			(at 49.53 126.5548 90)
 			(effects
 				(font
@@
 		)
 	)
+	(global_label "ramp_up_opto"
+		(shape output)
+		(at 114.3 52.07 90)
+		(fields_autoplaced yes)
+		(effects
+			(font
+				(size 1.27 1.27)
+			)
+			(justify left)
+		)
+		(property "Intersheetrefs" "${INTERSHEET_REFS}"
+			(at 114.3 35.9014 90)
+			(effects
+				(font
+					(size 1.27 1.27)
+				)
+				(justify left)
+				(hide yes)
+			)
+		)
+	)
 	(global_label "+VIN"
 		(shape output)
@@
 		)
 	)
+	(global_label "spare_opto"
+		(shape input)
+		(at 120.65 46.99 90)
+		(fields_autoplaced yes)
+		(effects
+			(font
+				(size 1.27 1.27)
+			)
+			(justify left)
+		)
+		(property "Intersheetrefs" "${INTERSHEET_REFS}"
+			(at 120.65 33.6636 90)
+			(effects
+				(font
+					(size 1.27 1.27)
+				)
+				(justify left)
+				(hide yes)
+			)
+		)
+	)
 	(global_label "GPIO_5"
 		(shape output)
@@
 		)
 	)
+	(global_label "spare_opto"
+		(shape output)
+		(at 120.65 29.21 0)
+		(fields_autoplaced yes)
+		(effects
+			(font
+				(size 1.27 1.27)
+			)
+			(justify left)
+		)
+		(property "Intersheetrefs" "${INTERSHEET_REFS}"
+			(at 133.9764 29.21 0)
+			(effects
+				(font
+					(size 1.27 1.27)
+				)
+				(justify left)
+				(hide yes)
+			)
+		)
+	)
 	(global_label "+3.3V"
 		(shape input)
@@
 	(global_label "+VOUT"
 		(shape output)
-		(at 194.31 147.32 0)
+		(at 198.12 147.32 0)
 		(fields_autoplaced yes)
 		(effects
@@
 		)
 		(property "Intersheetrefs" "${INTERSHEET_REFS}"
-			(at 203.5848 147.32 0)
+			(at 207.3948 147.32 0)
 			(effects
 				(font
@@
 	(symbol
 		(lib_id "custom_library:reset_fuse")
-		(at 180.34 147.32 0)
+		(at 184.15 147.32 0)
 		(unit 1)
 		(exclude_from_sim no)
@@
 		(fields_autoplaced yes)
 		(property "Reference" "RF2"
-			(at 179.705 140.97 0)
+			(at 183.515 140.97 0)
 			(effects
 				(font
@@
 		)
 		(property "Value" "~"
-			(at 179.705 143.51 0)
+			(at 183.515 143.51 0)
 			(effects
 				(font
@@
 		)
 		(property "Footprint" "footprints:PTC_RESET_FUSE"
-			(at 180.34 147.32 0)
+			(at 184.15 147.32 0)
 			(effects
 				(font
@@
 		)
 		(property "Datasheet" ""
-			(at 180.34 147.32 0)
+			(at 184.15 147.32 0)
 			(effects
 				(font
@@
 		)
 		(property "Description" ""
-			(at 180.34 147.32 0)
+			(at 184.15 147.32 0)
 			(effects
 				(font

Commit message: update
Parts:
- removed J2: 1757255, footprints:PHOENIX_1757255, symbol 1757255:1757255
- added J2: jst-power, footprints:PHOENIX_1757255, symbol custom_library:jst-power
- added J5: 1770979, footprints:PHOENIX_1770979, symbol 1770979:1770979
Connections:
- net +24V: no longer C1.1, C2.1, D1.2, J4.2, PS1.22 (+VIN), RF1.1, RF1.2
- net +3.3V: now also J5.3_1, J5.3_2, J5.4_1, J5.4_2
- net +VOUT: no longer RF2.2, U1.J2-19 (EXT_5V)
- net -Vin: now also J2.03
- net sim_home: now also J2.01
- net GPIO_19: now reaches U1.J3-8 (IO19)
- net GPIO_19: now also J5.1_1, J5.1_2
- net GPIO_18: now reaches U1.J3-9 (IO18)
- net GPIO_18: now also J5.2_1, J5.2_2
- new net +24V-Sim: D1.2, J2.02
- new net +VIN: C1.1, C2.1, PS1.22 (+VIN), RF1.2
- new net +VIN-dc: J4.2, RF1.1
- new net +VOUT-esp: RF2.2, U1.J2-19 (EXT_5V)
- no-connect marks 33 -> 31
