File: board_MKIV/board_MKIV.kicad_pcb (KiCad board)
At the start: 2 copper layers, 83.4 x 77.2 mm, 33 parts, among them J1 A-DF_09_A_KG-T4S, J2 jst-power, J3 JST -SM, J4 S3B-EH, J5 1770979, U1 ESP32-DEVKITC-32D, U2 LTV-846S

Commit message: update
Parts:
- added C1: UHE2A470MPD, footprints:PCAP_10x12_5-THRU-ELECT_NCA, F.Cu at (339.0, 125.0)
- added C1: UHE2A470MPD, footprints:PCAP_10x12_5-THRU-ELECT_NCA, F.Cu at (107.2, 166.6)
- added C2: UHE2A470MPD, footprints:PCAP_10x12_5-THRU-ELECT_NCA, F.Cu at (119.0, 166.6)
- added C2: UHE2A470MPD, footprints:PCAP_10x12_5-THRU-ELECT_NCA, F.Cu at (350.7, 125.0)
- added C3: 1000pf/3kV, footprints:CAPC3216X180N, F.Cu at (114.5, 104.7)
- added C3: 1000pf/3kV, footprints:CAPC3216X180N, B.Cu at (347.8, 145.0)
- added C4: ECA1HM100, footprints:CAPPRD200W50D500H1100, F.Cu at (111.0, 94.2)
- added C5: WCAP-ATG5_5X11, footprints:WCAP-ATG5_5X11_DXL_, F.Cu at (95.0, 94.1)
- added D1: SS34B-HF, footprints:DO214AASMB_CIP-L, F.Cu at (64.0, 85.8)
- added D1: SS34B-HF, footprints:DO214AASMB_CIP-L, B.Cu at (322.0, 138.0)
- added J1: 1757242, footprints:PHOENIX_1757242, F.Cu at (86.1, 68.5)
- added J2: jst-power, footprints:PHOENIX_1757255, F.Cu at (72.7, 68.5)
- added J3: JST -SM, footprints:CONN_BM04B-SRSS-TB_SPK, B.Cu at (373.0, 112.1)
- added J4: S3B-EH, footprints:CONN_S3B-EH_JST, F.Cu at (119.8, 75.3)
- added J4: S3B-EH, footprints:CONN_S3B-EH_JST, F.Cu at (324.1, 130.8)
- added J5: 1770979, footprints:PHOENIX_1770979, F.Cu at (402.8, 94.2)
- added J6: 20_pin_90, footprints:20_pin_90, F.Cu at (58.7, 125.6)
- added J7: 20-pin-straight, footprints:20_pin_straight, F.Cu at (58.4, 161.8)
- added PS1: REC5A-2405SW_H2, footprints:CONV_REC5A-2405SW_H2, F.Cu at (69.5, 175.2)
- added PS1: REC5A-2405SW_H2, footprints:CONV_REC5A-2405SW_H2, F.Cu at (341.3, 144.6)
- added R1: CRGH1206J4K7, footprints:RESC3115X65N, F.Cu at (53.5, 97.6)
- added R1: CRGH1206J4K7, footprints:RESC3115X65N, B.Cu at (334.5, 93.1)
- added R10: CR1206-FX-1002ELF, footprints:RESC3216X75N, B.Cu at (369.2, 126.2)
- added R11: CR1206-FX-1002ELF, footprints:RESC3216X75N, B.Cu at (376.4, 135.8)
- added R12: CR1206-FX-1002ELF, footprints:RESC3216X75N, B.Cu at (369.2, 135.7)
- added R13: CR1206-FX-1002ELF, footprints:RESC3216X75N, B.Cu at (376.4, 143.8)
- added R14: CR1206-FX-1002ELF, footprints:RESC3216X75N, B.Cu at (369.2, 143.8)
- added R15: CR1206-FX-1002ELF, footprints:RESC3216X75N, B.Cu at (369.2, 151.2)
- added R16: CR1206-FX-1002ELF, footprints:RESC3216X75N, B.Cu at (376.4, 151.2)
- added R17: CR1206-FX-1002ELF, footprints:RESC3216X75N, B.Cu at (377.0, 118.9)
- added R18: CR1206-FX-1002ELF, footprints:RESC3216X75N, B.Cu at (369.2, 118.9)
- added R19: ERJP08J105V, footprints:RES_ERJP08J105V, F.Cu at (79.5, 103.0)
- added R2: CRGH1206J4K7, footprints:RESC3115X65N, F.Cu at (58.0, 97.6)
- added R2: CRGH1206J4K7, footprints:RESC3115X65N, B.Cu at (330.0, 93.1)
- added R20: CRG1206F470R, footprints:RESC3115X65N, F.Cu at (93.5, 101.3)
- added R21: ERJP08J334V, footprints:RES_ERJP08J334V, F.Cu at (95.0, 105.5)
- added R22: ERJP08J105V, footprints:RES_ERJP08J105V, F.Cu at (79.5, 107.5)
- added R3: CRGH1206J4K7, footprints:RESC3115X65N, F.Cu at (62.3, 97.7)
- added R3: CRGH1206J4K7, footprints:RESC3115X65N, B.Cu at (332.4, 101.6)
- added R4: CRGH1206J4K7, footprints:RESC3015X65N, F.Cu at (66.8, 97.7)
- added R4: CRGH1206J4K7, footprints:RESC3015X65N, B.Cu at (332.4, 106.1)
- added R5: CRGH1206J4K7, footprints:RESC3115X65N, F.Cu at (71.0, 97.7)
- added R5: CRGH1206J4K7, footprints:RESC3115X65N, B.Cu at (332.4, 110.3)
- added R6: CRGH1206J4K7, footprints:RESC3115X65N, F.Cu at (75.5, 97.7)
- added R6: CRGH1206J4K7, footprints:RESC3115X65N, B.Cu at (332.4, 114.8)
- added R7: CRGH1206J4K7, footprints:RESC3115X65N, B.Cu at (328.0, 121.0)
- added R8: CRGH1206J4K7, footprints:RESC3115X65N, B.Cu at (331.5, 124.5)
- added R9: CR1206-FX-1002ELF, footprints:RESC3216X75N, B.Cu at (376.4, 126.3)
- added RF1: ~, footprints:PTC_RESET_FUSE, F.Cu at (124.1, 83.3)
- added RF1: ~, footprints:PTC_RESET_FUSE, F.Cu at (321.5, 146.1)
- added RF2: ~, footprints:PTC_RESET_FUSE, F.Cu at (349.3, 164.2)
- added RF2: ~, footprints:PTC_RESET_FUSE, F.Cu at (98.0, 133.8)
- added S1: DRR3016, footprints:DRR3010, F.Cu at (385.7, 149.4)
- added S1: DRR3016, footprints:DRR3010, B.Cu at (135.8, 71.7)
- added U1: ESP32-DEVKITC-32D, footprints:MODULE_ESP32-DEVKITC-32D, F.Cu at (372.9, 114.8)
- added U1: ESP32-DEVKITC-32D, footprints:MODULE_ESP32-DEVKITC-32D, B.Cu at (118.0, 170.8)
- added U2: LTV-846S, footprints:SOIC254P1016X460-16N, F.Cu at (62.8, 109.8)
- added U2: LTV-846S, footprints:SOIC254P1016X460-16N, B.Cu at (344.5, 112.0)
- added U3: TLV272CDR, footprints:D8, F.Cu at (103.4, 105.1)
- added U4: BAT46W, footprints:SOD123F, F.Cu at (103.8, 100.1)
- added U5: BA&, footprints:TO252-3_ROM, F.Cu at (103.7, 88.0)
- J1: value A-DF_09_A_KG-T4S -> 1757242; footprint footprints:ASSMANN_A-DF_09_A_KG-T4S -> footprints:PHOENIX_1757242
- moved C1 257.7 mm to (379.9, 34.1)
- moved C2 257.7 mm to (391.6, 34.1)
- moved C3 257.7 mm to (388.7, 54.1)
- moved D1 257.7 mm to (362.9, 47.1)
- moved J2 257.7 mm to (346.6, 47.0)
- moved J3 257.7 mm to (413.9, 21.2)
- moved J4 257.7 mm to (365.0, 39.8)
- moved J5 257.7 mm to (392.8, 0.15)
- moved PS1 257.7 mm to (382.1, 53.7)
- moved R1 257.7 mm to (375.4, 2.14)
- moved R10 257.7 mm to (410.1, 35.3)
- moved R11 257.7 mm to (417.3, 44.9)
- moved R12 257.7 mm to (410.1, 44.8)
- moved R13 257.7 mm to (417.3, 52.9)
- moved R14 257.7 mm to (410.1, 52.9)
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Connections:
- C3 pad 1: ESP_GND2 -> ESP_GND_signal
- J2 pad 01: sim_home -> sim_home_signal
- J2 pad 03: -Vin -> -Vin_signal
- J5 pad 4_1: ESP_GND2 -> +3.3V
- J5 pad 4_2: ESP_GND2 -> +3.3V
- PS1 pad 16: ESP_GND2 -> ESP_GND_signal
- RF2 pad 2: +VOUT-esp -> +VOUT_esp_signal
Routing:
- net +3.3V: track 217.6 -> 365.2 mm, vias 2 -> 4
- net ESP_GND2: track 190.1 -> 309.5 mm, vias 2 -> 4
- net GPIO_16: track 55.9 -> 111.8 mm
- net GPIO_5: track 55.5 -> 111.0 mm
- net GPIO_17: track 49.2 -> 98.5 mm, vias 2 -> 4
- net GPIO_4: track 42.2 -> 84.4 mm, vias 1 -> 2
- net GPIO_22: track 39.8 -> 79.7 mm
- net GPIO_26: track 32.8 -> 65.5 mm, vias 1 -> 2
- net GPIO_21: track 32.8 -> 65.5 mm
- net GPIO_25: track 28.6 -> 57.2 mm, vias 1 -> 2
- net GPIO_32: track 23.6 -> 47.2 mm, vias 1 -> 2
- net GPIO_33: track 15.6 -> 31.2 mm, vias 1 -> 2
- net /+24V-Sim: vias 8 -> 16
- net +VOUT-esp: vias 3 -> 6
- net +24V: vias 3 -> 6
Other:
- board size 83.4 x 77.2 mm -> 382.4 x 192.2 mm
- board text added: "CRGH1206J4K7"

Commit message: board update
Parts:
- removed the C1 at (339.0, 125.0)
- removed the C1 at (379.9, 34.1)
- removed the C2 at (350.7, 125.0)
- removed the C2 at (391.6, 34.1)
- removed the C3 at (347.8, 145.0)
- removed the C3 at (388.7, 54.1)
- removed the D1 at (362.9, 47.1)
- removed the D1 at (322.0, 138.0)
- removed the J1 at (357.5, 20.6)
- removed the J2 at (346.6, 47.0)
- removed the J3 at (413.9, 21.2)
- removed the J3 at (373.0, 112.1)
- removed J4 (x3): S3B-EH, footprints:CONN_S3B-EH_JST
- removed the J5 at (402.8, 94.2)
- removed the J5 at (392.8, 0.15)
- removed the PS1 at (341.3, 144.6)
- removed the PS1 at (382.1, 53.7)
- removed the R1 at (334.5, 93.1)
- removed the R1 at (375.4, 2.14)
- removed the R10 at (410.1, 35.3)
- removed the R10 at (369.2, 126.2)
- removed the R11 at (417.3, 44.9)
- removed the R11 at (376.4, 135.8)
- removed the R12 at (410.1, 44.8)
- removed the R12 at (369.2, 135.7)
- removed the R13 at (376.4, 143.8)
- removed the R13 at (417.3, 52.9)
- removed the R14 at (369.2, 143.8)
- removed the R14 at (410.1, 52.9)
- removed the R15 at (369.2, 151.2)
- removed the R15 at (410.1, 60.3)
- removed the R16 at (417.3, 60.3)
- removed the R16 at (376.4, 151.2)
- removed the R17 at (377.0, 118.9)
- removed the R17 at (417.9, 28.0)
- removed the R18 at (410.1, 28.0)
- removed the R18 at (369.2, 118.9)
- removed the R2 at (370.9, 2.14)
- removed the R2 at (330.0, 93.1)
- removed the R3 at (332.4, 101.6)
- removed the R3 at (373.3, 10.7)
- removed the R4 at (373.3, 15.2)
- removed the R4 at (332.4, 106.1)
- removed the R5 at (373.3, 19.4)
- removed the R5 at (332.4, 110.3)
- removed the R6 at (373.3, 23.9)
- removed the R6 at (332.4, 114.8)
- removed R7 (x2), R8 (x2): CRGH1206J4K7, footprints:RESC3115X65N
- removed the R9 at (417.3, 35.4)
- removed the R9 at (376.4, 126.3)
- removed the RF1 at (362.4, 55.2)
- removed the RF1 at (321.5, 146.1)
- removed the RF2 at (349.3, 164.2)
- removed the RF2 at (402.1, 61.1)
- removed S1 (x3): DRR3016, footprints:DRR3010
- removed the U1 at (372.9, 114.8)
- removed the U1 at (413.8, 23.9)
- removed the U2 at (344.5, 112.0)
- removed the U2 at (385.3, 21.1)
- added J3: JST -SM, footprints:CONN_BM04B-SRSS-TB_SPK, F.Cu at (134.0, 105.1)
- added J5: 1770979, footprints:PHOENIX_1770979, F.Cu at (129.0, 99.7)
- added R10: CR1206-FX-1002ELF, footprints:RESC3216X75N, F.Cu at (125.1, 97.1)
- added R11: CR1206-FX-1002ELF, footprints:RESC3216X75N, F.Cu at (125.1, 100.5)
- added R12: CR1206-FX-1002ELF, footprints:RESC3216X75N, F.Cu at (125.1, 103.8)
- added R13: CR1206-FX-1002ELF, footprints:RESC3216X75N, F.Cu at (125.1, 107.1)
- added R14: CR1206-FX-1002ELF, footprints:RESC3216X75N, F.Cu at (125.1, 110.4)
- added R15: CR1206-FX-1002ELF, footprints:RESC3216X75N, F.Cu at (125.1, 113.7)
- added R16: CR1206-FX-1002ELF, footprints:RESC3216X75N, F.Cu at (125.1, 117.1)
- added R17: CR1206-FX-1002ELF, footprints:RESC3216X75N, F.Cu at (125.1, 120.4)
- added R18: CR1206-FX-1002ELF, footprints:RESC3216X75N, F.Cu at (125.1, 123.7)
- added R9: CR1206-FX-1002ELF, footprints:RESC3216X75N, F.Cu at (125.1, 93.8)
- added S2: PB400EEQR1BLK, footprints:SW_PB400EEQR1BLK, F.Cu at (52.4, 171.8)
- added U6: SH-7070TB, footprints:SH-7070TB_7P1X7P3_NDC, B.Cu at (82.7, 175.3)
- C3, D1: moved to B.Cu
- moved RF1 111.4 mm to (50.6, 166.9)
- moved D1 93.4 mm to (52.3, 178.5)
- moved C3 84.5 mm to (69.0, 175.8), turned to 90 degrees
- moved RF2 60.0 mm to (58.4, 178.9), turned to -90 degrees
- moved C2 10.5 mm to (111.3, 173.8), turned to 90 degrees
- moved C1 10.4 mm to (99.8, 173.8), turned to 90 degrees
- moved PS1 7.00 mm to (76.5, 175.8)
- moved J6 3.67 mm to (59.7, 129.1)
- moved J7 1.87 mm to (60.2, 161.4)
- moved U1 1.60 mm to (119.7, 170.7)
Connections:
- C3 pad 1: (no net) -> ESP_GND2
- C3 pad 2: (no net) -> -Vin
- D1 pad 1: (no net) -> +24V
- D1 pad 2: (no net) -> /+24V-Sim
- J2 pad 03: -Vin_signal -> -Vin
- J6 pad A1: GPIO_19 -> GPIO_18
- J6 pad A10: unconnected-(J6-PadA10) -> GPIO_32
- J6 pad A2: GPIO_18 -> GPIO_19
- J6 pad A3: +3.3V -> GPIO_21
- J6 pad A4: unconnected-(J6-PadA4) -> GPIO_22
- J6 pad A5: unconnected-(J6-PadA5) -> GPIO_23
- J6 pad A6: unconnected-(J6-PadA6) -> GPIO_25
- J6 pad A7: unconnected-(J6-PadA7) -> GPIO_26
- J6 pad A8: unconnected-(J6-PadA8) -> GPIO_27
- J6 pad A9: unconnected-(J6-PadA9) -> GPIO_33
- J6 pad B1: +VOUT-esp -> unconnected-(J6-PadB1)
- J6 pad B10: sim_home -> +3.3V
- J6 pad B2: ESP_GND2 -> unconnected-(J6-PadB2)
- J6 pad B3: unconnected-(J6-PadB3) -> -Vin
- J6 pad B4: +VIN-dc -> +24V
- J6 pad B5: -Vin -> +VOUT_esp_signal
- J6 pad B7: spare -> +VIN-dc
- J6 pad B8: ramp_down -> unconnected-(J6-PadB8)
- J6 pad B9: ramp_up -> ESP_GND2
- J7 pad 1: sim_home_signal -> -Vin
- J7 pad 10: +VOUT_esp_signal -> GPIO_21
- J7 pad 11: unconnected-(J7-Pad11) -> +24V
- J7 pad 12: unconnected-(J7-Pad12) -> +VIN-dc
- J7 pad 13: unconnected-(J7-Pad13) -> +VOUT_esp_signal
- J7 pad 18: +3.3V -> ESP_GND2
- J7 pad 2: ramp_up_signal -> GPIO_27
- J7 pad 3: ramp_down_signal -> GPIO_26
- J7 pad 4: spare_signal -> GPIO_25
- J7 pad 5: unconnected-(J7-Pad5) -> GPIO_33
- J7 pad 6: -Vin_signal -> GPIO_32
- J7 pad 7: +VIN-dc -> +3.3V
- J7 pad 8: unconnected-(J7-Pad8) -> GPIO_23
- J7 pad 9: ESP_GND_signal -> GPIO_22
- PS1 pad 11: (no net) -> unconnected-(PS1-NC1-Pad11)
- PS1 pad 14: (no net) -> /+VOUT
- PS1 pad 16: (no net) -> ESP_GND2
- PS1 pad 2: (no net) -> -Vin
- PS1 pad 22: (no net) -> /+VIN
- PS1 pad 23: (no net) -> unconnected-(PS1-+VIN__1-Pad23)
- PS1 pad 3: (no net) -> unconnected-(PS1--VIN__1-Pad3)
- PS1 pad 9: (no net) -> unconnected-(PS1-NC-Pad9)
- RF1 pad 1: (no net) -> +VIN-dc
- RF1 pad 2: (no net) -> /+VIN
- RF2 pad 1: (no net) -> /+VOUT
- RF2 pad 2: (no net) -> +VOUT_esp_signal
- U1 pad J2-1: (no net) -> +3.3V
- U1 pad J2-10: (no net) -> GPIO_26
- U1 pad J2-11: (no net) -> GPIO_27
- U1 pad J2-12: (no net) -> unconnected-(U1-IO14-PadJ2-12)
- U1 pad J2-13: (no net) -> unconnected-(U1-IO12-PadJ2-13)
- U1 pad J2-14: (no net) -> ESP_GND2
- U1 pad J2-15: (no net) -> unconnected-(U1-IO13-PadJ2-15)
- U1 pad J2-16: (no net) -> unconnected-(U1-SD2-PadJ2-16)
- U1 pad J2-17: (no net) -> unconnected-(U1-SD3-PadJ2-17)
- U1 pad J2-18: (no net) -> unconnected-(U1-CMD-PadJ2-18)
- U1 pad J2-19: (no net) -> +VOUT_esp_signal
- U1 pad J2-2: (no net) -> unconnected-(U1-EN-PadJ2-2)
- U1 pad J2-3: (no net) -> unconnected-(U1-SENSOR_VP-PadJ2-3)
- U1 pad J2-4: (no net) -> unconnected-(U1-SENSOR_VN-PadJ2-4)
- U1 pad J2-5: (no net) -> unconnected-(U1-IO34-PadJ2-5)
- U1 pad J2-6: (no net) -> unconnected-(U1-IO35-PadJ2-6)
- U1 pad J2-7: (no net) -> GPIO_32
- U1 pad J2-8: (no net) -> GPIO_33
- U1 pad J2-9: (no net) -> GPIO_25
- U1 pad J3-1: (no net) -> ESP_GND2
- U1 pad J3-10: (no net) -> GPIO_5
- U1 pad J3-11: (no net) -> GPIO_17
- U1 pad J3-12: (no net) -> GPIO_16
- U1 pad J3-13: (no net) -> GPIO_4
- U1 pad J3-14: (no net) -> unconnected-(U1-IO0-PadJ3-14)
- U1 pad J3-15: (no net) -> unconnected-(U1-IO2-PadJ3-15)
- U1 pad J3-16: (no net) -> unconnected-(U1-IO15-PadJ3-16)
- U1 pad J3-17: (no net) -> unconnected-(U1-SD1-PadJ3-17)
- U1 pad J3-18: (no net) -> unconnected-(U1-SD0-PadJ3-18)
- U1 pad J3-19: (no net) -> unconnected-(U1-CLK-PadJ3-19)
- U1 pad J3-2: (no net) -> GPIO_23
- U1 pad J3-3: (no net) -> GPIO_22
- U1 pad J3-4: (no net) -> unconnected-(U1-TXD0-PadJ3-4)
- U1 pad J3-5: (no net) -> unconnected-(U1-RXD0-PadJ3-5)
- U1 pad J3-6: (no net) -> GPIO_21
- U1 pad J3-7: (no net) -> ESP_GND2
- U1 pad J3-8: (no net) -> GPIO_19
- U1 pad J3-9: (no net) -> GPIO_18
- U2 pad 10: GPIO_32 -> GPIO_32_
- U2 pad 12: GPIO_33 -> GPIO_33_
- U2 pad 14: GPIO_25 -> GPIO_25_
- U2 pad 16: GPIO_26 -> GPIO_26_
Routing:
- net +3.3V: track 365.2 -> 102.4 mm, vias 4 -> 1
- net ESP_GND2: track 309.5 -> 48.2 mm, vias 4 -> 0
- net GPIO_18: track 144.7 -> 40.1 mm
- net GPIO_19: track 143.7 -> 39.2 mm
- net GPIO_27: track 0.00 -> 70.7 mm
- net GPIO_23: track 0.00 -> 63.1 mm
- net GPIO_16: track 111.8 -> 49.5 mm, vias 0 -> 2
- net GPIO_5: track 111.0 -> 55.4 mm, vias 0 -> 2
- net GPIO_33: track 31.2 -> 71.2 mm, vias 2 -> 0
- net GPIO_17: track 98.5 -> 60.7 mm, vias 4 -> 2
- net +VOUT_esp_signal: track 0.00 -> 37.8 mm
- net GPIO_32: track 47.2 -> 70.7 mm, vias 2 -> 0
- net GPIO_22: track 79.7 -> 57.3 mm
- net GPIO_4: track 84.4 -> 64.2 mm
- net GPIO_21: track 65.5 -> 46.4 mm
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- added copper zone on B.Cu, net /+VIN
- removed copper zone on B.Cu, net +24V
- removed copper zone on F.Cu, net +24V
- removed copper zone on B.Cu, net +VIN-dc
- removed copper zone on B.Cu, net +VOUT-esp
- removed copper zone on F.Cu, net +VOUT-esp
- removed copper zone on B.Cu, net /+24V-Sim
- removed copper zone on F.Cu, net /+24V-Sim
- removed copper zone on F.Cu, net /+VIN
- removed copper zone on B.Cu, net /+VOUT
- removed copper zone on F.Cu, net /+VOUT
- removed copper zone on B.Cu, net /ramp_down_opto
- removed copper zone on F.Cu, net /ramp_down_opto
- removed copper zone on B.Cu, net /sim_home_opto
- removed copper zone on F.Cu, net /sim_home_opto
- removed copper zone on B.Cu, net GPIO_25
- removed copper zone on B.Cu, net GPIO_26
- removed copper zone on B.Cu, net GPIO_32
- removed copper zone on B.Cu, net GPIO_33
- removed copper zone on B.Cu, net ramp_down
- removed copper zone on F.Cu, net ramp_down
- removed copper zone on B.Cu, net ramp_up
- removed copper zone on F.Cu, net ramp_up
- removed copper zone on B.Cu, net ramp_up_opto
- removed copper zone on B.Cu, net sim_home
- removed copper zone on F.Cu, net sim_home
- removed copper zone on B.Cu, net spare
- removed copper zone on F.Cu, net spare
- removed copper zone on B.Cu, net spare_opto
- removed copper zone on F.Cu, net spare_opto
Other:
- board size 382.4 x 192.2 mm -> 100 x 120 mm
- board text removed: "Mark III"
- board text removed: "Sim Monitor"
