File: board_MKIV/board_MKIV.kicad_pcb (KiCad board)
At the start: 2 copper layers, 100 x 120 mm, 42 parts, among them J1 1757242, J2 jst-power, J3 JST -SM, J5 1770979, J6 20_pin_90, J7 20-pin-straight, U1 ESP32-DEVKITC-32D, U2 LTV-846S, U3 TLV272CDR, U4 BAT46W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

Commit message: update
Parts:
- added S1: DS01C-254-S-03BE, footprints:SW_DS01C-254-S-03BE, F.Cu at (128.7, 170.4)
- moved J6 3.72 mm to (60.2, 125.4)
- moved U1 0.56 mm to (120.0, 171.1)
- moved C1 0.45 mm to (99.3, 173.8)
- moved PS1 0.42 mm to (76.1, 175.8)
- moved RF1 0.23 mm to (50.6, 167.2)
- moved RF2 0.10 mm to (58.3, 178.9)
Connections:
- D1 pad 2: /+24V-Sim -> +VIN
- J2 pad 02: /+24V-Sim -> +24V
- J6 pad A1: GPIO_18 -> +VIN
- J6 pad A10: GPIO_32 -> CLK
- J6 pad A2: GPIO_19 -> +VIN-dc
- J6 pad A3: GPIO_21 -> +VOUT_esp_signal
- J6 pad A4: GPIO_22 -> GPIO_ANAG_34
- J6 pad A5: GPIO_23 -> unconnected-(J6-PadA5)
- J6 pad A6: GPIO_25 -> GPIO_ANAG_35
- J6 pad A7: GPIO_26 -> GPIO_13
- J6 pad A8: GPIO_27 -> ESP_GND2
- J6 pad A9: GPIO_33 -> GPIO_2
- J6 pad B1: unconnected-(J6-PadB1) -> GPIO_27
- J6 pad B10: +3.3V -> GPIO_21
- J6 pad B2: unconnected-(J6-PadB2) -> GPIO_26
- J6 pad B3: -Vin -> GPIO_25
- J6 pad B4: +24V -> GPIO_33
- J6 pad B5: +VOUT_esp_signal -> GPIO_32
- J6 pad B6: unconnected-(J6-PadB6) -> -Vin
- J6 pad B7: +VIN-dc -> +3.3V
- J6 pad B8: unconnected-(J6-PadB8) -> GPIO_23
- J6 pad B9: ESP_GND2 -> GPIO_22
- J7 pad 14: unconnected-(J7-Pad14) -> GPIO_ANAG_34
- J7 pad 16: unconnected-(J7-Pad16) -> GPIO_ANAG_35
- J7 pad 17: unconnected-(J7-Pad17) -> GPIO_13
- J7 pad 19: GPIO_18 -> GPIO_2
- J7 pad 20: GPIO_19 -> CLK
- U1 pad J2-12: unconnected-(U1-IO14-PadJ2-12) -> GPIO_14
- U1 pad J2-15: unconnected-(U1-IO13-PadJ2-15) -> GPIO_13
- U1 pad J2-5: unconnected-(U1-IO34-PadJ2-5) -> GPIO_ANAG_34
- U1 pad J2-6: unconnected-(U1-IO35-PadJ2-6) -> GPIO_ANAG_35
- U1 pad J3-15: unconnected-(U1-IO2-PadJ3-15) -> GPIO_2
- U1 pad J3-19: unconnected-(U1-CLK-PadJ3-19) -> CLK
Routing:
- net GPIO_ANAG_34: track 0.00 -> 116.0 mm, vias 0 -> 1
- net GPIO_ANAG_35: track 0.00 -> 111.3 mm, vias 0 -> 1
- net GPIO_13: track 0.00 -> 72.5 mm
- net +VOUT_esp_signal: track 37.1 -> 77.8 mm
- net GPIO_2: track 0.00 -> 28.2 mm
- net GPIO_18: track 40.1 -> 13.2 mm
- net GPIO_19: track 39.2 -> 14.6 mm
- net +3.3V: track 102.4 -> 127.0 mm
- net GPIO_27: track 49.3 -> 73.4 mm
- net GPIO_14: track 0.00 -> 23.1 mm
- net GPIO_26: track 51.3 -> 74.3 mm
- net GPIO_25: track 53.3 -> 75.2 mm
- net +VIN: track 73.9 -> 94.2 mm
- net /+24V-Sim: track 19.2 -> 0.00 mm
- net GPIO_32: track 56.0 -> 73.9 mm
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- added copper zone on B.Cu, net +VIN
- removed copper zone on B.Cu, net +24V
Other:
- outline, holes or cut-outs redrawn

Commit message: update
Parts:
- R1, R10, R11, R12, R13, R14, R15, R16, R19, R2, R22, R3, R4, R5, R6, R9, U2: moved to B.Cu
- moved R10 78.6 mm to (57.3, 57.4), turned to 90 degrees
- moved R9 74.0 mm to (60.6, 57.4), turned to 90 degrees
- moved R12 74.0 mm to (56.8, 75.3), turned to 90 degrees
- moved R11 69.7 mm to (60.1, 75.3), turned to 90 degrees
- moved R14 60.1 mm to (73.4, 141.1), turned to 180 degrees
- moved R15 58.2 mm to (76.5, 145.8), turned to -90 degrees
- moved R13 57.8 mm to (73.4, 133.0), turned to 180 degrees
- moved R22 55.6 mm to (79.0, 51.9), turned to -90 degrees
- moved R16 55.4 mm to (73.4, 137.1), turned to 180 degrees
- moved R18 52.4 mm to (138.1, 73.0), turned to 90 degrees
- moved R19 51.2 mm to (82.2, 51.9), turned to -90 degrees
- moved R17 48.4 mm to (134.8, 73.0), turned to 90 degrees
- moved U2 45.2 mm to (69.6, 65.1), turned to 180 degrees
- moved C3 41.6 mm to (66.0, 134.4)
- moved R6 40.3 mm to (80.4, 57.7), turned to 180 degrees
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Connections:
- R10 pad 1: GPIO_33_ -> GPIO_33
- R11 pad 1: GPIO_26_ -> GPIO_26
- R12 pad 1: GPIO_25_ -> GPIO_25
- R9 pad 1: GPIO_32_ -> GPIO_32
- U2 pad 10: GPIO_32_ -> GPIO_32
- U2 pad 12: GPIO_33_ -> GPIO_33
- U2 pad 14: GPIO_25_ -> GPIO_25
- U2 pad 16: GPIO_26_ -> GPIO_26
Routing:
- net GPIO_16: track 49.5 -> 74.0 mm
- net GPIO_5: track 55.3 -> 70.3 mm
- net GPIO_4: track 64.2 -> 69.8 mm
- net GPIO_17: track 60.7 -> 66.0 mm
- net +VOUT_esp_signal: track 77.8 -> 77.3 mm
Other:
- board size 100 x 120 mm -> 100 x 113.8 mm

Commit message: update
Parts:
- added LED1: COM-16347, footprints:COM-16347_SPK, B.Cu at (66.7, 140.2)
- added R7: CRL1206-FW-R330ELF, footprints:RESC3216X70N, B.Cu at (113.7, 147.6)
- R20, R21, U3, U4, U5: moved to B.Cu
- R22: value ERJP08J105V -> CRG1206F470R; footprint footprints:RES_ERJP08J105V -> footprints:RESC3115X65N
- moved R12 139.8 mm to (196.2, 86.4), turned to 180 degrees
- moved R11 136.3 mm to (196.2, 83.1), turned to 180 degrees
- moved R10 124.3 mm to (178.3, 85.9), turned to 180 degrees
- moved R1 121.2 mm to (200.6, 62.7), turned to -90 degrees
- moved R9 120.3 mm to (178.3, 82.6), turned to 180 degrees
- moved R2 116.2 mm to (196.1, 62.7), turned to -90 degrees
- moved R3 111.5 mm to (191.7, 62.7), turned to -90 degrees
- moved R4 106.9 mm to (187.2, 62.8), turned to -90 degrees
- moved R5 102.6 mm to (183.1, 62.8), turned to -90 degrees
- moved R6 98.3 mm to (178.6, 62.8), turned to -90 degrees
- moved R22 80.9 mm to (158.6, 66.7), turned to 0 degrees
- moved U2 69.2 mm to (135.2, 87.4), turned to -90 degrees
- moved R20 59.7 mm to (154.9, 61.2), turned to 90 degrees
- moved J1 34.9 mm to (68.0, 65.1)
- moved J2 34.2 mm to (88.3, 65.1)
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Connections:
- J2 pad 01: sim_home_signal -> sim_home
- J2 pad 02: +24V -> +VIN-dc
- R19 pad 1: sim_home_safe -> Net-(U3-1IN+)
- R19 pad 2: /sim_home_opto -> sim_home
- R20 pad 1: Net-(U3-1IN+) -> sim_home_safe
- R20 pad 2: sim_home -> /sim_home_opto
Routing:
- net -Vin: track 22.8 -> 96.8 mm
- net +VIN-dc: track 25.3 -> 92.6 mm
- net Net-(U3-1IN+): track 0.00 -> 54.4 mm, vias 0 -> 2
- net VDD: track 0.00 -> 23.7 mm
- net sim_home: track 0.00 -> 7.99 mm
- net Net-(LED1-DIN): track 0.00 -> 5.18 mm, vias 0 -> 1
- net GPIO_27: track 73.4 -> 76.5 mm
- net sim_home_safe: track 0.00 -> 1.27 mm
Other:
- board size 100 x 113.8 mm -> 100 x 84.6 mm

Commit message: update
Parts:
- J3: moved to B.Cu
- moved R7 47.8 mm to (66.3, 141.1)
- moved C3 18.4 mm to (82.4, 126.2), turned to 0 degrees
- moved R13 6.37 mm to (76.5, 127.5), turned to 90 degrees
- moved LED1 5.36 mm to (66.3, 134.9), turned to -90 degrees
- moved R16 2.81 mm to (73.7, 134.3)
- moved R14 1.99 mm to (73.7, 139.2)
- moved J3 1.80 mm to (159.0, 78.1)
Connections:
- net /+VOUT renamed /ESP-Board/+VOUT
- J7 pad 10: GPIO_21 -> -Vin
- J7 pad 6: -Vin -> +3.3V
- J7 pad 7: +3.3V -> GPIO_23
- J7 pad 8: GPIO_23 -> GPIO_22
- J7 pad 9: GPIO_22 -> GPIO_21
Routing:
- net -Vin: track 96.8 -> 74.0 mm
- net GPIO_27: track 76.5 -> 64.7 mm, vias 0 -> 1
- net ESP_GND2: track 52.6 -> 61.2 mm
- net GPIO_21: track 47.9 -> 50.5 mm
- net +VOUT_esp_signal: track 77.3 -> 79.6 mm
- net GPIO_23: track 68.0 -> 69.9 mm
- net Net-(LED1-DIN): track 5.18 -> 3.85 mm, vias 1 -> 0
- net GPIO_22: track 60.8 -> 61.9 mm
- net +3.3V: track 127.0 -> 128.1 mm
- net GPIO_4: track 69.8 -> 70.8 mm
- net GPIO_17: track 66.0 -> 66.9 mm

Commit message: MKIV Update
Parts:
- removed J5: 1770979, footprints:PHOENIX_1770979
- added ?: , , F.Cu at (146.4, 144.9)
- J3: moved to F.Cu
- R17, R18: moved to B.Cu
- moved J3 100.9 mm to (58.4, 85.6)
- moved R12 89.0 mm to (108.2, 99.5)
- moved R11 88.8 mm to (108.2, 95.0)
- moved J1 78.5 mm to (145.1, 79.5)
- moved R18 77.3 mm to (68.8, 107.3)
- moved R1 76.2 mm to (139.4, 108.2), turned to 180 degrees
- moved R9 74.6 mm to (108.2, 108.1)
- moved R10 72.4 mm to (108.2, 103.9)
- moved R17 70.7 mm to (73.0, 107.3)
- moved R2 69.9 mm to (139.4, 103.7), turned to 180 degrees
- moved R3 63.5 mm to (139.5, 98.9), turned to 180 degrees
- moved R4 57.3 mm to (139.4, 94.4), turned to 180 degrees
- moved R5 55.8 mm to (131.7, 84.8)
- moved R6 55.8 mm to (127.2, 84.8)
- moved R22 44.1 mm to (118.3, 84.8), turned to -90 degrees
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Connections:
- J1 pad 01: ramp_down_signal -> ramp_up
- J1 pad 02: ramp_up_signal -> ramp_down
Routing:
- net +3.3V: track 128.1 -> 266.4 mm, vias 1 -> 4
- net ESP_GND2: track 61.2 -> 147.0 mm, vias 0 -> 1
- net -Vin: track 74.0 -> 155.4 mm, vias 0 -> 1
- net GPIO_22: track 61.9 -> 137.3 mm, vias 0 -> 2
- net GPIO_26: track 74.3 -> 143.4 mm, vias 0 -> 1
- net GPIO_21: track 50.5 -> 118.7 mm, vias 0 -> 2
- net GPIO_25: track 75.2 -> 140.5 mm, vias 0 -> 1
- net GPIO_33: track 74.5 -> 138.1 mm, vias 0 -> 1
- net GPIO_32: track 73.9 -> 132.5 mm, vias 0 -> 1
- net sim_home_safe: track 1.27 -> 35.6 mm, vias 0 -> 2
- net ramp_up_opto: track 0.00 -> 22.2 mm
- net ramp_up: track 0.00 -> 20.6 mm
- net ramp_down: track 0.00 -> 20.2 mm
- net /ramp_down_opto: track 0.00 -> 19.5 mm
- net spare_opto: track 0.00 -> 18.1 mm
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Other:
- board size 100 x 84.6 mm -> 100.2 x 68.6 mm
- board text added: "1 2 3"
- board text added: "ID"
- board text added: "Mark IV"
- board text added: "Role Selection"
- board text added: "Sim Monitor"
