File: board_MKIV/_autosave-board_MKIV.kicad_pcb (KiCad board)
At the start: 2 copper layers, 100 x 120 mm, 42 parts, among them J1 1757242, J2 jst-power, J3 JST -SM, J5 1770979, J6 20_pin_90, J7 20-pin-straight, U1 ESP32-DEVKITC-32D, U2 LTV-846S, U3 TLV272CDR, U4 BAT46W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

Commit message: update
Connections:
- J7 pad 14: unconnected-(J7-Pad14) -> GPIO_2
- J7 pad 15: unconnected-(J7-Pad15) -> CLK
- J7 pad 16: unconnected-(J7-Pad16) -> GPIO_14
- J7 pad 17: unconnected-(J7-Pad17) -> GPIO_13
- U1 pad J2-12: unconnected-(U1-IO14-PadJ2-12) -> GPIO_14
- U1 pad J2-15: unconnected-(U1-IO13-PadJ2-15) -> GPIO_13
- U1 pad J2-6: unconnected-(U1-IO35-PadJ2-6) -> GPIO_ANAG_35
- U1 pad J3-15: unconnected-(U1-IO2-PadJ3-15) -> GPIO_2
- U1 pad J3-19: unconnected-(U1-CLK-PadJ3-19) -> CLK
Routing:
- net GPIO_18: track 40.1 -> 0.00 mm
- net GPIO_19: track 39.2 -> 0.02 mm
Changed lines of the file:
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@@
 	(net 18 "+VIN")
 	(net 19 "unconnected-(U1-SENSOR_VN-PadJ2-4)")
-	(net 20 "unconnected-(U1-CLK-PadJ3-19)")
+	(net 20 "GPIO_13")
 	(net 21 "unconnected-(U1-SD1-PadJ3-17)")
 	(net 22 "unconnected-(U1-TXD0-PadJ3-4)")
 	(net 23 "unconnected-(U1-SD0-PadJ3-18)")
-	(net 24 "unconnected-(U1-IO13-PadJ2-15)")
+	(net 24 "GPIO_2")
 	(net 25 "GPIO_32_")
 	(net 26 "unconnected-(U1-IO34-PadJ2-5)")
 	(net 27 "unconnected-(U1-CMD-PadJ2-18)")
 	(net 28 "unconnected-(U1-IO0-PadJ3-14)")
-	(net 29 "unconnected-(U1-IO2-PadJ3-15)")
+	(net 29 "CLK")
 	(net 30 "unconnected-(U1-SENSOR_VP-PadJ2-3)")
 	(net 31 "unconnected-(U1-RXD0-PadJ3-5)")
@@
 	(net 36 "unconnected-(U1-IO15-PadJ3-16)")
 	(net 37 "GPIO_22")
-	(net 38 "unconnected-(U1-IO35-PadJ2-6)")
+	(net 38 "GPIO_14")
 	(net 39 "unconnected-(U1-EN-PadJ2-2)")
 	(net 40 "+24V")
-	(net 41 "unconnected-(U1-IO14-PadJ2-12)")
+	(net 41 "GPIO_ANAG_35")
 	(net 42 "GPIO_32")
 	(net 43 "GPIO_33")
@@
 	(net 70 "unconnected-(J6-PadB1)")
 	(net 71 "unconnected-(J6-PadB6)")
-	(net 72 "unconnected-(J7-Pad17)")
-	(net 73 "unconnected-(J7-Pad16)")
-	(net 74 "unconnected-(J7-Pad15)")
-	(net 75 "unconnected-(J7-Pad14)")
 	(footprint "footprints:RESC3115X65N"
 		(layer "F.Cu")
@@
 			(layers "*.Cu" "*.Mask")
 			(remove_unused_layers no)
-			(net 75 "unconnected-(J7-Pad14)")
+			(net 24 "GPIO_2")
 			(pinfunction "14")
-			(pintype "unspecified+no_connect")
+			(pintype "unspecified")
 		)
 		(pad "15" thru_hole circle
@@
 			(layers "*.Cu" "*.Mask")
 			(remove_unused_layers no)
-			(net 74 "unconnected-(J7-Pad15)")
+			(net 29 "CLK")
 			(pinfunction "15")
-			(pintype "unspecified+no_connect")
+			(pintype "unspecified")
 		)
 		(pad "16" thru_hole circle
@@
 			(layers "*.Cu" "*.Mask")
 			(remove_unused_layers no)
-			(net 73 "unconnected-(J7-Pad16)")
+			(net 38 "GPIO_14")
 			(pinfunction "16")
-			(pintype "unspecified+no_connect")
+			(pintype "unspecified")
 		)
 		(pad "17" thru_hole circle
@@
 			(layers "*.Cu" "*.Mask")
 			(remove_unused_layers no)
-			(net 72 "unconnected-(J7-Pad17)")
+			(net 20 "GPIO_13")
 			(pinfunction "17")
-			(pintype "unspecified+no_connect")
+			(pintype "unspecified")
 		)
 		(pad "18" thru_hole circle
@@
 		(fp_text user "*"
 			(at -4.9276 4.3434 180)
+			(unlocked yes)
 			(layer "B.SilkS")
 			(effects
@@
 		(fp_text user "*"
 			(at -4.9276 4.3434 180)
-			(unlocked yes)
 			(layer "B.SilkS")
 			(effects
@@
 			)
 		)
-		(fp_text user "${REFERENCE}"
-			(at 0 0 180)
+		(fp_text user "*"
+			(at -3.175 3.5687 180)
 			(unlocked yes)
 			(layer "B.Fab")
@@
 			)
 		)
-		(fp_text user "*"
-			(at -3.175 3.5687 180)
+		(fp_text user "${REFERENCE}"
+			(at 0 0 180)
 			(unlocked yes)
 			(layer "B.Fab")
@@
 			(layers "*.Cu" "*.Mask")
 			(remove_unused_layers no)
-			(net 38 "unconnected-(U1-IO35-PadJ2-6)")
+			(net 41 "GPIO_ANAG_35")
 			(pinfunction "IO35")
-			(pintype "bidirectional+no_connect")
+			(pintype "bidirectional")
 			(solder_mask_margin 0.102)
 		)
@@
 			(layers "*.Cu" "*.Mask")
 			(remove_unused_layers no)
-			(net 41 "unconnected-(U1-IO14-PadJ2-12)")
+			(net 38 "GPIO_14")
 			(pinfunction "IO14")
-			(pintype "bidirectional+no_connect")
+			(pintype "bidirectional")
 			(solder_mask_margin 0.102)
 		)
@@
 			(layers "*.Cu" "*.Mask")
 			(remove_unused_layers no)
-			(net 24 "unconnected-(U1-IO13-PadJ2-15)")
+			(net 20 "GPIO_13")
 			(pinfunction "IO13")
-			(pintype "bidirectional+no_connect")
+			(pintype "bidirectional")
 			(solder_mask_margin 0.102)
 		)
@@
 			(layers "*.Cu" "*.Mask")
 			(remove_unused_layers no)
-			(net 29 "unconnected-(U1-IO2-PadJ3-15)")
+			(net 24 "GPIO_2")
 			(pinfunction "IO2")
-			(pintype "bidirectional+no_connect")
+			(pintype "bidirectional")
 			(solder_mask_margin 0.102)
 		)
@@
 			(layers "*.Cu" "*.Mask")
 			(remove_unused_layers no)
-			(net 20 "unconnected-(U1-CLK-PadJ3-19)")
+			(net 29 "CLK")
 			(pinfunction "CLK")
-			(pintype "input+no_connect")
+			(pintype "input")
 			(solder_mask_margin 0.102)
 		)
@@
 	)
 	(segment
-		(start 83.375 159.1375)
-		(end 120.5675 159.1375)
-		(width 0.254)
-		(layer "F.Cu")
-		(net 51)
-	)
-	(segment
-		(start 120.5675 159.1375)
-		(end 121.705 158)
-		(width 0.254)
-		(layer "F.Cu")
-		(net 51)
-	)
-	(segment
 		(start 83.075 158.8375)
-		(end 83.375 159.1375)
+		(end 83.0875 158.85)
 		(width 0.254)
 		(layer "F.Cu")
@@
 	)
 	(segment
-		(start 80.535 158.8375)
-		(end 82.685 156.6875)
-		(width 0.254)
-		(layer "F.Cu")
-		(net 52)
-	)
-	(segment
-		(start 117.8525 156.6875)
-		(end 119.165 158)
-		(width 0.254)
-		(layer "F.Cu")
-		(net 52)
-	)
-	(segment
-		(start 82.685 156.6875)
-		(end 117.8525 156.6875)
-		(width 0.254)
-		(layer "F.Cu")
-		(net 52)
-	)
-	(segment
