File: board_MKIV/board_MKIV.kicad_sch (KiCad schematic)
At the start: 42 parts, among them J1 1757242, J2 jst-power, J3 JST -SM, J4 S3B-EH, J5 1770979, J6-Right-Angle 86094327313755E1LF, J7-Straight 86094328314755V1LF, U1 ESP32-DEVKITC-32D, U2 LTV-846S, U3 TLV272CDR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

Commit message: update
Parts:
- removed J6-Right-Angle: 86094327313755E1LF, 86094327313755E1LF:AMPHENOL_86094327313755E1LF, symbol 86094327313755E1LF:86094327313755E1LF
- removed J7-Straight: 86094328314755V1LF, 86094328314755V1LF:AMPHENOL_86094328314755V1LF, symbol 86094328314755V1LF:86094328314755V1LF
- added J6: 20_pin_90, CONN_XC5A-2022_OMR, symbol 20_pin_90:XC5A-2022
- added J7: 20-pin-straight, CONN_XC5B-2021_OMR, symbol 20_pin_straight:XC5B-2021
Connections:
- net +24V: no longer C5.1, U5.1 (INPUT)
- net +3.3V: now also J7.18
- net +VIN-dc: now also C5.1, U5.1 (INPUT), J7.7
- net +VOUT-esp: no longer RF2.2
- net -Vin: no longer J2.03
- net ESP_GND2: no longer C3.1, PS1.16 (-VOUT)
- net GPIO_18: now also J7.19
- net GPIO_19: now also J7.20
- net ramp_down: no longer J1.01
- net ramp_up: no longer J1.02
- net sim_home: no longer J2.01
- new net +VOUT_esp_signal: J7.10, RF2.2
- new net -Vin_signal: J2.03, J7.6
- new net ESP_GND_signal: C3.1, J7.9, PS1.16 (-VOUT)
- new net ramp_down_signal: J1.01, J7.3
- new net ramp_up_signal: J1.02, J7.2
- new net sim_home_signal: J2.01, J7.1
- new net spare_signal: J7.4
Other:
- moved on the sheet: C1, C2, C3, C4, C5, D1, J1, J2, J4, J5, PS1, RF1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

Commit message: board update
Parts:
- removed J4: S3B-EH, footprints:CONN_S3B-EH_JST, symbol custom_library:S3B-EH
- removed S1: DRR3016, footprints:DRR3010, symbol DRR3016:DRR3016
- added S2: PB400EEQR1BLK, footprints:SW_PB400EEQR1BLK, symbol PB400EEQR1BLK:PB400EEQR1BLK
- added U6: SH-7070TB, SH-7070TB_7P1X7P3_NDC, symbol rot_switch:SH-7070TB
- J1: footprint 1757242:PHOENIX_1757242 -> footprints:PHOENIX_1757242
- J6: footprint CONN_XC5A-2022_OMR -> footprints:20_pin_90
- J7: footprint CONN_XC5B-2021_OMR -> footprints:20_pin_straight
Connections:
- net +VOUT-esp is gone; now on net +VOUT_esp_signal: U1.J2-19 (EXT_5V)
- net spare_signal is gone; now on net GPIO_25: J7.4
- net +24V: now also J6.B4, J7.11, S2.1, S2.3
- net +3.3V: now also J6.B10, J7.7, U6.2, U6.5; no longer J7.18
- net +VIN-dc: now also J6.B7, J7.12, S2.2, S2.4; no longer J7.7
- net +VOUT_esp_signal: now also J6.B5, J7.13; no longer J7.10
- net -Vin: now also J2.03, J6.B3, J7.1
- net ESP_GND2: now also C3.1, J6.B9, J7.18, PS1.16 (-VOUT)
- net GPIO_16: now also U6.4
- net GPIO_17: now also U6.3
- net GPIO_18: now also J6.A1
- net GPIO_19: now also J6.A2
- net GPIO_21: now also J6.A3, J7.10
- net GPIO_22: now also J6.A4, J7.9
- net GPIO_25: now also J6.A6; no longer R12.1, U2.14
- net GPIO_26: now also J6.A7, J7.3; no longer R11.1, U2.16
- net GPIO_32: now also J6.A10, J7.6; no longer R9.1, U2.10
- net GPIO_33: now also J6.A9, J7.5; no longer R10.1, U2.12
- net GPIO_4: now also U6.1
- net GPIO_5: now also U6.6
- net ramp_down_signal: no longer J7.3
- net ramp_up_signal: no longer J7.2
- net sim_home_signal: no longer J7.1
- net GPIO_23: now reaches J6.A5
- net GPIO_23: now also J7.8, U1.J3-2 (IO23)
- net GPIO_27: now reaches J6.A8
- net GPIO_27: now also J7.2, U1.J2-11 (IO27)
- removed net -Vin_signal: J2.03, J7.6
- removed net ESP_GND_signal: C3.1, J7.9, PS1.16 (-VOUT)
- new net GPIO_25_: R12.1, U2.14
- new net GPIO_26_: R11.1, U2.16
- new net GPIO_32_: R9.1, U2.10
- new net GPIO_33_: R10.1, U2.12
- no-connect marks 26 -> 32
Other:
- moved on the sheet: J6, J7

Commit message: update
Parts:
- added S1: DS01C-254-S-03BE, DS01C-254-S-03BE:SW_DS01C-254-S-03BE, symbol DS01C-254-S-03BE:DS01C-254-S-03BE
Connections:
- net +24V: no longer J7.11
- net +VIN: now also J7.11, S2.2, S2.4
- net +VIN-dc: no longer S2.2, S2.4
- net -Vin: now also J7.6; no longer J7.1
- net GPIO_18: now also S1.2B; no longer J7.19
- net GPIO_19: now also S1.1B; no longer J7.20
- net GPIO_25: now also J7.3; no longer J7.4
- net GPIO_26: now also J7.2; no longer J7.3
- net GPIO_27: now also J7.1; no longer J7.2
- net GPIO_32: now also J7.5; no longer J7.6
- net GPIO_33: now also J7.4; no longer J7.5
- net GPIO_14: now reaches U1.J2-12 (IO14)
- net GPIO_14: now also J7.16, S1.3B
- net GPIO_13: now reaches U1.J2-15 (IO13)
- net GPIO_13: now also J7.17
- net GPIO_2: now reaches U1.J3-15 (IO2)
- net GPIO_2: now also J7.14
- net CLK: now reaches U1.J3-19 (CLK)
- net CLK: now also J7.15
- no-connect marks 32 -> 24

Commit message: update
Parts:
- S1: footprint DS01C-254-S-03BE:SW_DS01C-254-S-03BE -> footprints:SW_DS01C-254-S-03BE
- U6: footprint SH-7070TB_7P1X7P3_NDC -> footprints:SH-7070TB_7P1X7P3_NDC
Connections:
- net +24V: now also J2.02; no longer J6.B4
- net +3.3V: now also J6.B7, S1.1A, S1.2A, S1.3A; no longer J6.B10
- net +VIN: now also D1.2, J6.A1
- net +VIN-dc: now also J6.A2; no longer J6.B7
- net +VOUT_esp_signal: now also J6.A3; no longer J6.B5
- net -Vin: now also J6.B6; no longer J6.B3
- net CLK: now also J6.A10, J7.20; no longer J7.15
- net ESP_GND2: now also J6.A8; no longer J6.B9
- net GPIO_13: now also J6.A7
- net GPIO_14: now also S1.1B; no longer J7.16, S1.3B
- net GPIO_18: no longer J6.A1
- net GPIO_19: now also S1.3B; no longer J6.A2, S1.1B
- net GPIO_2: now also J6.A9, J7.19; no longer J7.14
- net GPIO_21: now also J6.B10; no longer J6.A3
- net GPIO_22: now also J6.B9; no longer J6.A4
- net GPIO_23: now also J6.B8; no longer J6.A5
- net GPIO_25: now also J6.B3; no longer J6.A6
- net GPIO_26: now also J6.B2; no longer J6.A7
- net GPIO_27: now also J6.B1; no longer J6.A8
- net GPIO_32: now also J6.B5; no longer J6.A10
- net GPIO_33: now also J6.B4; no longer J6.A9
- net GPIO_ANAG_34: now reaches U1.J2-5 (IO34)
- net GPIO_ANAG_34: now also J6.A4, J7.14
- net GPIO_ANAG_35: now reaches U1.J2-6 (IO35)
- net GPIO_ANAG_35: now also J6.A6, J7.16
- removed net +24V-Sim: D1.2, J2.02
- no-connect marks 24 -> 20
Other:
- moved on the sheet: D1, RF1

Commit message: update
Connections:
- net GPIO_25_ is gone; now on net GPIO_25: R12.1, U2.14
- net GPIO_26_ is gone; now on net GPIO_26: R11.1, U2.16
- net GPIO_32_ is gone; now on net GPIO_32: R9.1, U2.10
- net GPIO_33_ is gone; now on net GPIO_33: R10.1, U2.12
Changed lines of the file:
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@@
 		)
 	)
-	(global_label "GPIO_25_"
+	(global_label "GPIO_25"
 		(shape output)
 		(at 308.61 67.31 0)
@@
 		)
 		(property "Intersheetrefs" "${INTERSHEET_REFS}"
-			(at 320.4247 67.31 0)
+			(at 319.4571 67.31 0)
 			(effects
 				(font
@@
 		)
 	)
-	(global_label "GPIO_32_"
+	(global_label "GPIO_32"
 		(shape output)
 		(at 295.91 46.99 0)
@@
 		)
 		(property "Intersheetrefs" "${INTERSHEET_REFS}"
-			(at 307.7247 46.99 0)
+			(at 306.7571 46.99 0)
 			(effects
 				(font
@@
 		)
 	)
-	(global_label "GPIO_26_"
+	(global_label "GPIO_26"
 		(shape output)
 		(at 295.91 77.47 0)
@@
 		)
 		(property "Intersheetrefs" "${INTERSHEET_REFS}"
-			(at 307.7247 77.47 0)
+			(at 306.7571 77.47 0)
 			(effects
 				(font
@@
 		)
 	)
-	(global_label "GPIO_33_"
+	(global_label "GPIO_33"
 		(shape output)
 		(at 308.61 57.15 0)
@@
 		)
 		(property "Intersheetrefs" "${INTERSHEET_REFS}"
-			(at 320.4247 57.15 0)
-			(effects
-				(font
+			(at 319.4571 57.15 0)
+			(effects
+				(font

Commit message: update
Parts:
- removed R22: ERJP08J105V, footprints:RES_ERJP08J105V, symbol ERJP08J105V:ERJP08J105V
- added LED1: COM-16347, footprints:COM-16347_SPK, symbol RGB_LED:COM-16347
- added R22: CRG1206F470R, footprints:RESC3115X65N, symbol CRG1206F470R:CRG1206F470R
- added R7: CRL1206-FW-R330ELF, footprints:RESC3216X70N, symbol CRL1206-FW-R330ELF:CRL1206-FW-R330ELF
Connections:
- net sim_home_signal is gone; now on net sim_home: J2.01
- net +24V: no longer J2.02
- net +VIN-dc: now also J2.02
- net +VOUT_esp_signal: now also LED1.1 (VDD)
- net ESP_GND2: now also LED1.3 (VSS)
- net GPIO_27: now also LED1.2 (DOUT), R7.2
- net sim_home: now also R19.2; no longer R20.2
- net sim_home_opto: now also R20.2, R22.2; no longer R19.2
- net sim_home_safe: now also R20.1, R22.1; no longer R19.1
- net at R21.2, U3.3 (1IN+), U4.2: now also R19.1; no longer R20.1
- new net: LED1.4 (DIN), R7.1
Other:
- moved on the sheet: R19, R20

Commit message: update
Parts:
- removed C1, C2: UHE2A470MPD, footprints:PCAP_10x12_5-THRU-ELECT_NCA, symbol custom_library:UHE2A470MPD
- removed C3: 1000pf/3kV, footprints:CAPC3216X180N, symbol CL31B106KAHNNNE:CL31B106KAHNNNE
- removed D1: SS34B-HF, footprints:DO214AASMB_CIP-L, symbol custom_library:SS34B-HF
- removed J7: 20-pin-straight, footprints:20_pin_straight, symbol 20_pin_straight:XC5B-2021
- removed LED1: COM-16347, footprints:COM-16347_SPK, symbol RGB_LED:COM-16347
- removed PS1: REC5A-2405SW_H2, footprints:CONV_REC5A-2405SW_H2, symbol custom_library:REC5A-2405SW_H2
- removed R13, R14, R15, R16: CR1206-FX-1002ELF, footprints:RESC3216X75N, symbol CR1206-FX-1002ELF:CR1206-FX-1002ELF
- removed R7: CRL1206-FW-R330ELF, footprints:RESC3216X70N, symbol CRL1206-FW-R330ELF:CRL1206-FW-R330ELF
- removed RF1, RF2: ~, footprints:PTC_RESET_FUSE, symbol custom_library:reset_fuse
- removed S1: DS01C-254-S-03BE, footprints:SW_DS01C-254-S-03BE, symbol DS01C-254-S-03BE:DS01C-254-S-03BE
- removed S2: PB400EEQR1BLK, footprints:SW_PB400EEQR1BLK, symbol PB400EEQR1BLK:PB400EEQR1BLK
- removed U1: ESP32-DEVKITC-32D, footprints:MODULE_ESP32-DEVKITC-32D, symbol custom_library:ESP32-DEVKITC-32D
- removed U6: SH-7070TB, footprints:SH-7070TB_7P1X7P3_NDC, symbol rot_switch:SH-7070TB
Connections:
- no-connect marks 20 -> 4
Other:
- added sheet ESP-Board (ESP-Board.kicad_sch)
- moved on the sheet: J1, J2, J3, J5, J6, R1, R10, R11, R12, R17, R18, R2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

Commit message: MKIV Update
Parts:
- removed J5: 1770979, footprints:PHOENIX_1770979, symbol 1770979:1770979
Connections:
- net ramp_down_signal is gone; now on net ramp_up: J1.01
- net ramp_up_signal is gone; now on net ramp_down: J1.02
- net +3.3V: now also J6.B6; no longer J6.B7
- net -Vin: now also J6.B10; no longer J6.B6
- net GPIO_21: now also J6.B9; no longer J6.B10
- net GPIO_22: now also J6.B8; no longer J6.B9
- net GPIO_23: now also J6.B7; no longer J6.B8
